File: kicad/macrolev.kicad_pcb (KiCad board)
At the start: 2 copper layers, 3 parts, among them U1 RP2040, U2 A1101ELHL

Commit message: 🚧  Pcb in progress
Parts:
- removed D1: 1.5KExxA, Diode_THT:D_DO-201AE_P15.24mm_Horizontal
- added AM0:1: ESC, void_switch:VoidSwitch_1u_SMD, F.Cu at (157.2, 154.0)
- added AM0:10: Z, void_switch:VoidSwitch_1u_SMD, F.Cu at (200.0, 211.1)
- added AM0:11: 2, void_switch:VoidSwitch_1u_SMD, F.Cu at (195.3, 154.0)
- added AM0:12: W, void_switch:VoidSwitch_1u_SMD, F.Cu at (204.8, 173.0)
- added AM0:13: LAlt, void_switch:VoidSwitch_1.25u_SMD, F.Cu at (207.2, 230.2)
- added AM0:14: S, void_switch:VoidSwitch_1u_SMD, F.Cu at (209.6, 192.1)
- added AM0:15: 3, void_switch:VoidSwitch_1u_SMD, F.Cu at (214.3, 154.0)
- added AM0:16: E, void_switch:VoidSwitch_1u_SMD, F.Cu at (223.8, 173.0)
- added AM0:2: Tab, void_switch:VoidSwitch_1.5u_SMD, F.Cu at (161.9, 173.0)
- added AM0:3: CAPS, void_switch:VoidSwitch_1.75u_SMD, F.Cu at (164.3, 192.1)
- added AM0:4: LShift, void_switch:VoidSwitch_1.25u_SMD, F.Cu at (159.5, 211.1)
- added AM0:5: LCtrl, void_switch:VoidSwitch_1.25u_SMD, F.Cu at (159.5, 230.2)
- added AM0:6: 1, void_switch:VoidSwitch_1u_SMD, F.Cu at (176.2, 154.0)
- added AM0:7: Super, void_switch:VoidSwitch_1.25u_SMD, F.Cu at (183.4, 230.2)
- added AM0:8: Q, void_switch:VoidSwitch_1u_SMD, F.Cu at (185.7, 173.0)
- added AM0:9: A, void_switch:VoidSwitch_1u_SMD, F.Cu at (190.5, 192.1)
- added AM1:1: X, void_switch:VoidSwitch_1u_SMD, F.Cu at (219.1, 211.1)
- added AM1:10: T, void_switch:VoidSwitch_1u_SMD, F.Cu at (261.9, 173.0)
- added AM1:11: G, void_switch:VoidSwitch_1u_SMD, F.Cu at (266.7, 192.1)
- added AM1:12: B, void_switch:VoidSwitch_1u_SMD, F.Cu at (276.2, 211.1)
- added AM1:13: 6, void_switch:VoidSwitch_1u_SMD, F.Cu at (271.5, 154.0)
- added AM1:14: Y, void_switch:VoidSwitch_1u_SMD, F.Cu at (281.0, 173.0)
- added AM1:15: H, void_switch:VoidSwitch_1u_SMD, F.Cu at (285.8, 192.1)
- added AM1:2: D, void_switch:VoidSwitch_1u_SMD, F.Cu at (228.6, 192.1)
- added AM1:3: C, void_switch:VoidSwitch_1u_SMD, F.Cu at (238.1, 211.1)
- added AM1:4: 4, void_switch:VoidSwitch_1u_SMD, F.Cu at (233.4, 154.0)
- added AM1:5: R, void_switch:VoidSwitch_1u_SMD, F.Cu at (242.9, 173.0)
- added AM1:6: F, void_switch:VoidSwitch_1u_SMD, F.Cu at (247.7, 192.1)
- added AM1:7: V, void_switch:VoidSwitch_1u_SMD, F.Cu at (257.2, 211.1)
- added AM1:8: LSpace, void_switch:VoidSwitch_1.75u_SMD, F.Cu at (235.7, 230.2)
- added AM1:9: 5, void_switch:VoidSwitch_1u_SMD, F.Cu at (252.4, 154.0)
- added AM2:1: RSpace, void_switch:VoidSwitch_1.75u_SMD, F.Cu at (307.2, 230.2)
- added AM2:10: Comma, void_switch:VoidSwitch_1u_SMD, F.Cu at (333.4, 211.1)
- added AM2:11: 9, void_switch:VoidSwitch_1u_SMD, F.Cu at (328.6, 154.0)
- added AM2:12: O, void_switch:VoidSwitch_1u_SMD, F.Cu at (338.1, 173.0)
- added AM2:2: N, void_switch:VoidSwitch_1u_SMD, F.Cu at (295.3, 211.1)
- added AM2:3: 7, void_switch:VoidSwitch_1u_SMD, F.Cu at (290.5, 154.0)
- added AM2:4: U, void_switch:VoidSwitch_1u_SMD, F.Cu at (300.0, 173.0)
- added AM2:5: J, void_switch:VoidSwitch_1u_SMD, F.Cu at (304.8, 192.1)
- added AM2:6: M, void_switch:VoidSwitch_1u_SMD, F.Cu at (314.3, 211.1)
- added AM2:7: 8, void_switch:VoidSwitch_1u_SMD, F.Cu at (309.6, 154.0)
- added AM2:8: I, void_switch:VoidSwitch_1u_SMD, F.Cu at (319.1, 173.0)
- added AM2:9: K, void_switch:VoidSwitch_1u_SMD, F.Cu at (323.9, 192.1)
- added AM3:1: RAlt, void_switch:VoidSwitch_1.25u_SMD, F.Cu at (335.8, 230.2)
- added AM3:10: LBrack, void_switch:VoidSwitch_1u_SMD, F.Cu at (376.2, 173.0)
- added AM3:11: Quot, void_switch:VoidSwitch_1u_SMD, F.Cu at (381.0, 192.1)
- added AM3:12: Equal, void_switch:VoidSwitch_1u_SMD, F.Cu at (385.8, 154.0)
- added AM3:13: RBrack, void_switch:VoidSwitch_1u_SMD, F.Cu at (395.3, 173.0)
- added AM3:2: L, void_switch:VoidSwitch_1u_SMD, F.Cu at (342.9, 192.1)
- added AM3:3: Period, void_switch:VoidSwitch_1u_SMD, F.Cu at (352.4, 211.1)
- added AM3:4: Zero, void_switch:VoidSwitch_1u_SMD, F.Cu at (347.7, 154.0)
- added AM3:5: Fn, void_switch:VoidSwitch_1.25u_SMD, F.Cu at (359.6, 230.2)
- added AM3:6: P, void_switch:VoidSwitch_1u_SMD, F.Cu at (357.2, 173.0)
- added AM3:7: Semi, void_switch:VoidSwitch_1u_SMD, F.Cu at (361.9, 192.1)
- added AM3:8: Slash, void_switch:VoidSwitch_1u_SMD, F.Cu at (181.0, 211.1)
- added AM3:9: Minus, void_switch:VoidSwitch_1u_SMD, F.Cu at (366.7, 154.0)
- added AM4:1: RShift, void_switch:VoidSwitch_1.5u_SMD, F.Cu at (376.2, 211.1)
- added AM4:2: LEFT, void_switch:VoidSwitch_1u_SMD, F.Cu at (387.4, 236.5)
- added AM4:3: Enter, void_switch:VoidSwitch_1.75u_SMD, F.Cu at (407.2, 192.1)
- added AM4:4: BS, void_switch:VoidSwitch_1.5u_SMD, F.Cu at (409.6, 154.0)
- added AM4:5: Bslash, void_switch:VoidSwitch_1u_SMD, F.Cu at (414.3, 173.0)
- added AM4:6: UP, void_switch:VoidSwitch_1u_SMD, F.Cu at (406.4, 217.5)
- added AM4:7: DOWN, void_switch:VoidSwitch_1u_SMD, F.Cu at (406.4, 236.5)
- added AM4:8: RIGHT, void_switch:VoidSwitch_1u_SMD, F.Cu at (425.4, 236.5)
- added AMUX1: CD74HC4067SM, Package_SO:SSOP-24_5.3x8.2mm_P0.65mm, F.Cu at (195.2, 182.6)
- added AMUX2: CD74HC4067SM, Package_SO:SSOP-24_5.3x8.2mm_P0.65mm, F.Cu at (252.4, 182.6)
- added AMUX3: CD74HC4067SM, Package_SO:SSOP-24_5.3x8.2mm_P0.65mm, F.Cu at (328.5, 182.5)
- added AMUX4: CD74HC4067SM, Package_SO:SSOP-24_5.3x8.2mm_P0.65mm, F.Cu at (390.6, 182.6)
- added BOOT1: TS-1187A-B-A-B, footprint:SW-SMD_4P-L5.1-W5.1-P3.70-LS6.5-TL-2, F.Cu at (430.8, 219.1)
- added C1: 100nF, Capacitor_SMD:C_0402_1005Metric, F.Cu at (440.2, 206.5)
- added C10: 100nF, Capacitor_SMD:C_0402_1005Metric, F.Cu at (440.2, 207.5)
- added C11: 1uF, Capacitor_SMD:C_0402_1005Metric, F.Cu at (443.8, 194.9)
- added C12: 100nF, Capacitor_SMD:C_0402_1005Metric, F.Cu at (444.9, 201.8)
- added C13: 10uF, Capacitor_SMD:C_0402_1005Metric, F.Cu at (447.9, 188.2)
- added C14: 100nF, Capacitor_SMD:C_0402_1005Metric, F.Cu at (445.1, 198.2)
- added C15: 100nF, Capacitor_SMD:C_0402_1005Metric, F.Cu at (439.8, 194.9)
- added C17: 100nF, Capacitor_SMD:C_0402_1005Metric, F.Cu at (444.1, 197.2)
- added C18: 10uF, Capacitor_SMD:C_0402_1005Metric, F.Cu at (457.8, 196.7)
- added C19: 10uF, Capacitor_SMD:C_0402_1005Metric, F.Cu at (448.0, 196.7)
- added C2: 100nF, Capacitor_SMD:C_0402_1005Metric, F.Cu at (438.8, 194.9)
- added C20: 22pF, Capacitor_SMD:C_0402_1005Metric, F.Cu at (435.0, 206.9)
- added C21: 22pF, Capacitor_SMD:C_0402_1005Metric, F.Cu at (436.8, 212.4)
- added C3: 100nF, Capacitor_SMD:C_0402_1005Metric, F.Cu at (433.9, 198.2)
- added C4: 1uF, Capacitor_SMD:C_0402_1005Metric, F.Cu at (481.0, 157.4)
- added C5: 1uF, Capacitor_SMD:C_0402_1005Metric, F.Cu at (477.6, 157.4)
- added C6: 100nF, Capacitor_SMD:C_0402_1005Metric, F.Cu at (433.9, 202.1)
- added C7: 1uF, Capacitor_SMD:C_0402_1005Metric, F.Cu at (442.8, 194.9)
- added C8: 10uF, Capacitor_SMD:C_0402_1005Metric, F.Cu at (457.7, 188.2)
- added C9: 100nF, Capacitor_SMD:C_0402_1005Metric, F.Cu at (438.1, 188.8)
- added Debug1: Conn_01x05, Connector_PinHeader_2.54mm:PinHeader_1x05_P2.54mm_Vertical, F.Cu at (423.0, 207.9)
- added FID1: Fiducial, Fiducial:Fiducial_1mm_Mask3mm, F.Cu at (151.6, 148.4)
- added FID2: Fiducial, Fiducial:Fiducial_1mm_Mask3mm, F.Cu at (456.4, 149.2)
- added FID3: Fiducial, Fiducial:Fiducial_1mm_Mask3mm, F.Cu at (373.9, 241.3)
- added Flash1: W25Q128JVS, Package_SO:SOIC-8_5.23x5.23mm_P1.27mm, F.Cu at (432.5, 190.8)
- added LDO1: NCP1117-3.3_SOT223, Package_TO_SOT_SMD:SOT-223-3_TabPin2, F.Cu at (452.8, 190.9)
- added LDO2: NCP1117-3.3_SOT223, Package_TO_SOT_SMD:SOT-223-3_TabPin2, F.Cu at (452.9, 199.4)
- added MCU1: RP2040, footprint:LQFN-56_L7.0-W7.0-P0.4-EP, F.Cu at (439.4, 200.8)
- added R1: 10k, Resistor_SMD:R_0402_1005Metric, F.Cu at (439.4, 215.1)
- added R10: 10k, Resistor_SMD:R_0402_1005Metric, F.Cu at (445.1, 152.4)
- added R11: 1k, Resistor_SMD:R_0402_1005Metric, F.Cu at (438.6, 210.2)
- added R2: 10K, Resistor_SMD:R_0402_1005Metric, F.Cu at (474.6, 159.7)
- added R3: 10K, Resistor_SMD:R_0402_1005Metric, F.Cu at (474.6, 158.6)
- added R4: 1k, Resistor_SMD:R_0402_1005Metric, F.Cu at (427.4, 215.1)
- added R5: 10k, Resistor_SMD:R_0402_1005Metric, F.Cu at (426.6, 188.2)
- added R6: 27, Resistor_SMD:R_0402_1005Metric, F.Cu at (440.8, 194.9)
- added R7: 27, Resistor_SMD:R_0402_1005Metric, F.Cu at (441.8, 194.9)
- added R8: 10k, Resistor_SMD:R_0402_1005Metric, F.Cu at (440.9, 173.1)
- added R9: 10k, Resistor_SMD:R_0402_1005Metric, F.Cu at (443.1, 173.1)
- added RST1: TS-1187A-B-A-B, footprint:SW-SMD_4P-L5.1-W5.1-P3.70-LS6.5-TL-2, F.Cu at (442.7, 219.1)
- added SW1: RotaryEncoder_Switch, Rotary_Encoder:RotaryEncoder_Alps_EC11E-Switch_Vertical_H20mm, F.Cu at (439.6, 170.2)
- added TP1: In/Trig, TestPoint:TestPoint_Pad_D1.5mm, F.Cu at (474.6, 161.7)
- added TP2: +, TestPoint:TestPoint_Pad_D1.5mm, F.Cu at (485.0, 160.8)
- added TP3: -, TestPoint:TestPoint_Pad_1.5x1.5mm, F.Cu at (485.1, 158.2)
- added U10: GH39FKSW, Package_TO_SOT_SMD:SOT-23, F.Cu at (241.4, 214.4)
- added U11: GH39FKSW, Package_TO_SOT_SMD:SOT-23, F.Cu at (355.7, 214.4)
- added U12: GH39FKSW, Package_TO_SOT_SMD:SOT-23, F.Cu at (184.2, 214.4)
- added U13: GH39FKSW, Package_TO_SOT_SMD:SOT-23, F.Cu at (298.5, 214.4)
- added U14: GH39FKSW, Package_TO_SOT_SMD:SOT-23, F.Cu at (231.8, 195.3)
- added U15: GH39FKSW, Package_TO_SOT_SMD:SOT-23, F.Cu at (384.2, 195.3)
- added U16: GH39FKSW, Package_TO_SOT_SMD:SOT-23, F.Cu at (162.8, 233.4)
- added U17: GH39FKSW, Package_TO_SOT_SMD:SOT-23, F.Cu at (308.1, 195.3)
- added U18: GH39FKSW, Package_TO_SOT_SMD:SOT-23, F.Cu at (227.1, 176.3)
- added U19: GH39FKSW, Package_TO_SOT_SMD:SOT-23, F.Cu at (365.2, 195.3)
- added U20: GH39FKSW, Package_TO_SOT_SMD:SOT-23, F.Cu at (162.8, 214.4)
- added U21: GH39FKSW, Package_TO_SOT_SMD:SOT-23, F.Cu at (303.3, 176.3)
- added U22: GH39FKSW, Package_TO_SOT_SMD:SOT-23, F.Cu at (217.6, 157.2)
- added U23: GH39FKSW, Package_TO_SOT_SMD:SOT-23, F.Cu at (379.5, 176.3)
- added U24: GH39FKSW, Package_TO_SOT_SMD:SOT-23, F.Cu at (167.6, 195.3)
- added U25: GH39FKSW, Package_TO_SOT_SMD:SOT-23, F.Cu at (293.8, 157.2)
- added U26: GH39FKSW, Package_TO_SOT_SMD:SOT-23, F.Cu at (236.6, 157.2)
- added U27: GH39FKSW, Package_TO_SOT_SMD:SOT-23, F.Cu at (370.0, 157.2)
- added U28: GH39FKSW, Package_TO_SOT_SMD:SOT-23, F.Cu at (165.2, 176.3)
- added U29: GH39FKSW, Package_TO_SOT_SMD:SOT-23, F.Cu at (312.8, 157.2)
- added U3: GH39FKSW, Package_TO_SOT_SMD:SOT-23, F.Cu at (379.5, 214.4)
- added U30: GH39FKSW, Package_TO_SOT_SMD:SOT-23, F.Cu at (246.2, 176.3)
- added U31: GH39FKSW, Package_TO_SOT_SMD:SOT-23, F.Cu at (389.0, 157.2)
- added U32: GH39FKSW, Package_TO_SOT_SMD:SOT-23, F.Cu at (160.4, 157.2)
- added U33: GH39FKSW, Package_TO_SOT_SMD:SOT-23, F.Cu at (322.3, 176.3)
- added U34: GH39FKSW, Package_TO_SOT_SMD:SOT-23, F.Cu at (255.7, 157.2)
- added U35: GH39FKSW, Package_TO_SOT_SMD:SOT-23, F.Cu at (398.6, 176.3)
- added U36: GH39FKSW, Package_TO_SOT_SMD:SOT-23, F.Cu at (189.0, 176.3)
- added U37: GH39FKSW, Package_TO_SOT_SMD:SOT-23, F.Cu at (331.9, 157.2)
- added U38: GH39FKSW, Package_TO_SOT_SMD:SOT-23, F.Cu at (274.7, 157.2)
- added U39: GH39FKSW, Package_TO_SOT_SMD:SOT-23, F.Cu at (412.8, 157.2)
- added U4: GH39FKSW, Package_TO_SOT_SMD:SOT-23, F.Cu at (193.8, 195.3)
- added U40: GH39FKSW, Package_TO_SOT_SMD:SOT-23, F.Cu at (179.4, 157.2)
- added U41: GH39FKSW, Package_TO_SOT_SMD:SOT-23, F.Cu at (350.9, 157.2)
- added U42: GH39FKSW, Package_TO_SOT_SMD:SOT-23, F.Cu at (265.2, 176.3)
- added U43: GH39FKSW, Package_TO_SOT_SMD:SOT-23, F.Cu at (417.6, 176.3)
- added U44: GH39FKSW, Package_TO_SOT_SMD:SOT-23, F.Cu at (198.5, 157.2)
- added U45: GH39FKSW, Package_TO_SOT_SMD:SOT-23, F.Cu at (341.4, 176.3)
- added U46: GH39FKSW, Package_TO_SOT_SMD:SOT-23, F.Cu at (284.2, 176.3)
- added U47: GH39FKSW, Package_TO_SOT_SMD:SOT-23, F.Cu at (410.4, 195.3)
- added U48: GH39FKSW, Package_TO_SOT_SMD:SOT-23, F.Cu at (208.0, 176.3)
- added U49: GH39FKSW, Package_TO_SOT_SMD:SOT-23, F.Cu at (360.4, 176.3)
- added U5: GH39FKSW, Package_TO_SOT_SMD:SOT-23, F.Cu at (317.6, 214.4)
- added U50: GH39FKSW, Package_TO_SOT_SMD:SOT-23, F.Cu at (289.0, 195.3)
- added U51: GH39FKSW, Package_TO_SOT_SMD:SOT-23, F.Cu at (428.7, 239.8)
- added U52: GH39FKSW, Package_TO_SOT_SMD:SOT-23, F.Cu at (212.8, 195.3)
- added U53: GH39FKSW, Package_TO_SOT_SMD:SOT-23, F.Cu at (346.1, 195.3)
- added U54: GH39FKSW, Package_TO_SOT_SMD:SOT-23, F.Cu at (269.9, 195.3)
- added U55: GH39FKSW, Package_TO_SOT_SMD:SOT-23, F.Cu at (409.6, 220.7)
- added U56: GH39FKSW, Package_TO_SOT_SMD:SOT-23, F.Cu at (222.3, 214.4)
- added U57: GH39FKSW, Package_TO_SOT_SMD:SOT-23, F.Cu at (336.6, 214.4)
- added U58: GH39FKSW, Package_TO_SOT_SMD:SOT-23, F.Cu at (279.5, 214.4)
- added U59: GH39FKSW, Package_TO_SOT_SMD:SOT-23, F.Cu at (409.6, 239.8)
- added U6: GH39FKSW, Package_TO_SOT_SMD:SOT-23, F.Cu at (239.0, 233.4)
- added U60: GH39FKSW, Package_TO_SOT_SMD:SOT-23, F.Cu at (210.4, 233.4)
- added U61: GH39FKSW, Package_TO_SOT_SMD:SOT-23, F.Cu at (339.0, 233.4)
- added U62: GH39FKSW, Package_TO_SOT_SMD:SOT-23, F.Cu at (250.9, 195.3)
- added U63: GH39FKSW, Package_TO_SOT_SMD:SOT-23, F.Cu at (390.6, 239.8)
- added U64: GH39FKSW, Package_TO_SOT_SMD:SOT-23, F.Cu at (203.3, 214.4)
- added U65: GH39FKSW, Package_TO_SOT_SMD:SOT-23, F.Cu at (327.1, 195.3)
- added U7: GH39FKSW, Package_TO_SOT_SMD:SOT-23, F.Cu at (362.8, 233.4)
- added U8: GH39FKSW, Package_TO_SOT_SMD:SOT-23, F.Cu at (186.6, 233.4)
- added U9: GH39FKSW, Package_TO_SOT_SMD:SOT-23, F.Cu at (310.4, 233.4)
- added UART1: Conn_01x05, Connector_PinHeader_2.54mm:PinHeader_1x05_P2.54mm_Vertical, F.Cu at (428.7, 207.9)
- added USB1: Conn_01x04, Connector_PinHeader_2.54mm:PinHeader_1x04_P2.54mm_Vertical, F.Cu at (438.2, 183.9)
- added X1: 12MHz, footprint:OSC-SMD_4P-L3.2-W2.5-BL, F.Cu at (436.3, 209.5)
- U1: value RP2040 -> DRV2605LDGS; footprint Package_DFN_QFN:QFN-56-1EP_7x7mm_P0.4mm_EP3.2x3.2mm -> Package_SO:VSSOP-10_3x3mm_P0.5mm
- U2: value A1101ELHL -> GH39FKSW; footprint Package_TO_SOT_SMD:SOT-23W -> Package_TO_SOT_SMD:SOT-23
- moved U1 456.9 mm to (479.3, 159.7)
- moved U2 257.4 mm to (260.4, 214.4), turned to -45 degrees
Connections:
- U1 pad 1: Net-(U1-Pad1) -> Net-(C5-Pad1)
- U1 pad 10: Net-(U1-Pad1) -> +3.3V
- U1 pad 2: unconnected-(U1-Pad2) -> /SCL0
- U1 pad 3: unconnected-(U1-Pad3) -> /SDA0
- U1 pad 4: unconnected-(U1-Pad4) -> Net-(TP1-Pad1)
- U1 pad 5: unconnected-(U1-Pad5) -> +3.3V
- U1 pad 6: unconnected-(U1-Pad6) -> +3.3V
- U1 pad 7: unconnected-(U1-Pad7) -> Net-(TP2-Pad1)
- U1 pad 8: unconnected-(U1-Pad8) -> GND
- U1 pad 9: unconnected-(U1-Pad9) -> Net-(TP3-Pad1)
- U2 pad 1: unconnected-(U2-Pad1) -> +3.3VA
- U2 pad 2: unconnected-(U2-Pad2) -> /AMUX1:0
- U2 pad 3: unconnected-(U2-Pad3) -> GND
Routing:
- net +3.3V: track 0.00 -> 63.7 mm, vias 0 -> 1
- net /RUN: track 0.00 -> 50.5 mm, vias 0 -> 1
- net /QSPI_SS: track 0.00 -> 40.7 mm
- net /SWCLK: track 0.00 -> 31.8 mm, vias 0 -> 1
- net /SWD: track 0.00 -> 30.1 mm, vias 0 -> 1
- net /QSPI_SD1: track 0.00 -> 16.7 mm
- net /QSPI_SD2: track 0.00 -> 15.1 mm
- net /D-: track 0.00 -> 11.2 mm
- net /D+: track 0.00 -> 10.6 mm
- net /UART1_RTS: track 0.00 -> 8.80 mm
- net /QSPI_SD3: track 0.00 -> 8.49 mm
- net Net-(BOOT1-Pad1): track 0.00 -> 8.18 mm
- net /UART1_TX: track 0.00 -> 8.11 mm
- net /UART1_CTS: track 0.00 -> 7.91 mm
- net /XIN: track 0.00 -> 7.31 mm
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- added copper zone on B.Cu, net GND
- added copper zone on F.Cu, net GND
Other:
- board outline added: 312.7 x 101.6 mm

Commit message: 📝  Add wooting 60HE pictures
Parts:
- removed the C4 at (481.0, 157.4)
- removed the C5 at (477.6, 157.4)
- removed the R2 at (474.6, 159.7)
- removed the R3 at (474.6, 158.6)
- removed TP1: In/Trig, TestPoint:TestPoint_Pad_D1.5mm
- removed TP2: +, TestPoint:TestPoint_Pad_D1.5mm
- removed TP3: -, TestPoint:TestPoint_Pad_1.5x1.5mm
- removed the U1 at (479.3, 159.7)
- removed UART1: Conn_01x05, Connector_PinHeader_2.54mm:PinHeader_1x05_P2.54mm_Vertical
- moved BOOT1 3.09 mm to (432.8, 216.8)
- moved R2 3.09 mm to (429.5, 212.8)
- moved R1 2.31 mm to (439.4, 212.8)
- moved RST1 2.31 mm to (442.7, 216.8)
- moved C3 0.75 mm to (434.2, 197.5), turned to 90 degrees
- moved C12 0.69 mm to (445.5, 197.6), turned to 90 degrees
- moved C2 0.33 mm to (438.8, 194.6)
- renumbered C12 to C10, C13 to C11, C14 to C12, C15 to C13, C17 to C15, C18 to C16, C19 to C17, C20 to C18, C21 to C19, C6 to C4, C7 to C5, C8 to C6, C9 to C7, C10 to C8, C11 to C9, R4 to R2, R5 to R3, R6 to R4, R7 to R5, R11 to R6, R8 to R7, R9 to R8, R10 to R9, U2 to U1, U11 to U10, U12 to U11, U13 to U12, U14 to U13, U15 to U14, U16 to U15, U17 to U16, U18 to U17, U19 to U18, U20 to U19, U3 to U2, U21 to U20, U22 to U21, U23 to U22, U24 to U23, U25 to U24, U26 to U25, U27 to U26, U28 to U27, U29 to U28, U30 to U29, U4 to U3, U31 to U30, U32 to U31, U33 to U32, U34 to U33, U35 to U34, U36 to U35, U37 to U36, U38 to U37, U39 to U38, U40 to U39, U5 to U4, U41 to U40, U42 to U41, U43 to U42, U44 to U43, U45 to U44, U46 to U45, U47 to U46, U48 to U47, U49 to U48, U50 to U49, U6 to U5, U51 to U50, U52 to U51, U53 to U52, U54 to U53, U55 to U54, U56 to U55, U57 to U56, U58 to U57, U59 to U58, U60 to U59, U7 to U6, U61 to U60, U62 to U61, U63 to U62, U64 to U63, U65 to U64, U8 to U7, U9 to U8, U10 to U9
Routing:
- net +3.3VA: track 4.59 -> 1922.2 mm, vias 0 -> 75
- net /ADC0: track 0.00 -> 338.5 mm, vias 0 -> 2
- net /SELECT0: track 0.00 -> 311.2 mm, vias 0 -> 5
- net /SELECT1: track 0.00 -> 309.2 mm, vias 0 -> 5
- net /SELECT2: track 0.00 -> 301.9 mm, vias 0 -> 5
- net /SELECT3: track 0.00 -> 300.2 mm, vias 0 -> 5
- net /ADC1: track 0.00 -> 272.4 mm, vias 0 -> 2
- net /ADC2: track 0.00 -> 197.0 mm, vias 0 -> 2
- net /ADC3: track 0.00 -> 135.7 mm, vias 0 -> 2
- net +3.3V: track 63.7 -> 171.4 mm, vias 1 -> 4
- net /AMUX3:12: track 0.00 -> 71.9 mm
- net /ENC_SW: track 3.27 -> 68.8 mm, vias 0 -> 1
- net /AMUX0:3: track 0.00 -> 64.3 mm
- net /AMUX3:14: track 0.00 -> 62.7 mm
- net /AMUX3:1: track 0.00 -> 61.1 mm
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