File: kicad/macrolev.kicad_pcb (KiCad board)
At the start: 2 copper layers, 309.6 x 95.2 mm, 107 parts, among them J2 I2C, J3 DEBUG, J4 USBC, SW1 BOOT_BTN, SW2 RST_BTN, U1 A1101ELHL, U10 A1101ELHL, U11 A1101ELHL, U12 A1101ELHL, U13 A1101ELHL, U14 A1101ELHL, U15 A1101ELHL, U16 A1101ELHL, U17 A1101ELHL, U18 A1101ELHL, U19 A1101ELHL, U2 A1101ELHL, U20 A1101ELHL, U21 A1101ELHL, U22 A1101ELHL, U23 A1101ELHL, U24 A1101ELHL, U25 A1101ELHL, U26 A1101ELHL, U27 A1101ELHL, U28 A1101ELHL, U29 A1101ELHL, U3 A1101ELHL, U30 A1101ELHL, U31 A1101ELHL, U32 A1101ELHL, U33 A1101ELHL, U34 A1101ELHL, U35 A1101ELHL, U36 A1101ELHL, U37 A1101ELHL, U38 A1101ELHL, U39 A1101ELHL, U4 A1101ELHL, U40 A1101ELHL, U41 A1101ELHL, U42 A1101ELHL, U43 A1101ELHL, U44 A1101ELHL, U45 A1101ELHL, U46 A1101ELHL, U47 A1101ELHL, U48 A1101ELHL, U49 A1101ELHL, U5 A1101ELHL, U50 A1101ELHL, U51 A1101ELHL, U52 A1101ELHL, U53 A1101ELHL, U54 A1101ELHL, U55 A1101ELHL, U56 A1101ELHL, U57 A1101ELHL, U58 A1101ELHL, U59 A1101ELHL, U6 A1101ELHL, U60 A1101ELHL, U61 A1101ELHL, U62 A1101ELHL, U63 A1101ELHL, U64 A1101ELHL, U65 A1101ELHL, U66 A1101ELHL, U67 A1101ELHL, U68 AMS1117-3.3, U69 STM32F411CEU6, U7 A1101ELHL, U8 A1101ELHL, U9 A1101ELHL, Y1 25MHz/20ppm/15pF

Commit message: fix(pcb): apply feedback from PrintedCircuitBoard sub
Parts:
- removed J4: USBC, Connector_PinHeader_2.54mm:PinHeader_1x04_P2.54mm_Vertical
- added J1: USBC, Connector_PinHeader_2.54mm:PinHeader_1x04_P2.54mm_Vertical, B.Cu at (186.1, 47.2)
- added R1: 1.2K, Resistor_SMD:R_0402_1005Metric_Pad0.72x0.64mm_HandSolder, B.Cu at (173.5, 47.8)
- added R2: 1.2K, Resistor_SMD:R_0402_1005Metric_Pad0.72x0.64mm_HandSolder, B.Cu at (172.0, 49.6)
- SW1: value BOOT_BTN -> RST_BTN
- SW2: value RST_BTN -> BOOT_BTN
- moved D1 157.2 mm to (192.5, 54.9)
- moved R5 157.2 mm to (195.7, 54.9)
- moved SW2 139.3 mm to (175.9, 66.5), turned to -90 degrees
- moved R4 137.2 mm to (176.4, 62.1), turned to 0 degrees
- moved SW1 120.9 mm to (155.6, 54.5), turned to -90 degrees
- moved R3 119.8 mm to (156.1, 50.1), turned to 0 degrees
- moved C10 23.7 mm to (189.5, 51.5), turned to 0 degrees
- moved FB2 23.0 mm to (189.3, 49.8), turned to 180 degrees
- moved J2 21.6 mm to (184.1, 72.9), turned to 0 degrees
- moved Y1 19.9 mm to (161.6, 55.1), turned to 135 degrees
- moved C13 17.9 mm to (162.8, 52.2), turned to 135 degrees
- moved C12 17.6 mm to (164.4, 53.8), turned to -45 degrees
- moved C9 17.6 mm to (163.9, 49.4), turned to 135 degrees
- moved U68 16.1 mm to (183.2, 52.6), turned to 0 degrees
- moved C6 15.9 mm to (164.3, 48.3), turned to -45 degrees
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Routing:
- net /BOOT0: track 192.6 -> 22.3 mm, vias 4 -> 0
- net /NRST: track 181.1 -> 15.8 mm, vias 4 -> 0
- net +3.3V: track 256.0 -> 119.2 mm, vias 12 -> 8
- net /SELECT1: track 325.7 -> 446.3 mm, vias 8 -> 16
- net /SELECT0: track 329.9 -> 441.2 mm, vias 6 -> 16
- net /SELECT3: track 330.8 -> 441.4 mm, vias 8 -> 16
- net /SELECT2: track 334.8 -> 436.2 mm, vias 8 -> 16
- net /ADC2: track 61.0 -> 88.6 mm
- net /ADC3: track 130.4 -> 156.8 mm
- net /ADC1: track 34.4 -> 57.0 mm
- net /ADC4: track 170.0 -> 189.3 mm, vias 2 -> 0
- net /ADC0: track 97.1 -> 113.8 mm, vias 2 -> 0
- net /I2C_SCL: track 9.53 -> 26.1 mm
- net /I2C_SDA: track 12.8 -> 27.7 mm
- net GND: track 314.9 -> 302.2 mm, vias 95 -> 97
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- removed copper zone on F.Cu, net +3.3V
- removed copper zone on B.Cu, net +3.3VA
- removed copper zone on B.Cu, net +5V
- removed copper zone on B.Cu, net /VBUS

Commit message: change pcb routing
Parts:
- moved D1 7.30 mm to (191.9, 47.6)
- moved R5 7.30 mm to (195.1, 47.6)
- moved J3 6.64 mm to (185.7, 48.1)
- moved J1 2.68 mm to (185.7, 44.5)
- moved R3 1.15 mm to (157.2, 49.8), turned to -90 degrees
- moved C10 0.92 mm to (189.7, 52.5)
- moved C11 0.92 mm to (177.9, 54.7)
- moved U68 0.92 mm to (183.4, 53.5)
- moved FB2 0.52 mm to (189.5, 50.2)
- moved SW1 0.51 mm to (155.6, 54.0)
- moved C4 0.28 mm to (174.4, 45.0)
Routing:
- net GND: track 302.2 -> 38.5 mm, vias 97 -> 463
- net +3.3VA: track 2007.4 -> 2049.5 mm, vias 27 -> 26
- net +5V: track 10.4 -> 0.09 mm
- net +3.3V: track 119.2 -> 112.1 mm
- net /SELECT2: track 436.2 -> 442.1 mm, vias 16 -> 8
- net /SELECT3: track 441.4 -> 446.8 mm, vias 16 -> 8
- net /AMUX3:8: track 34.0 -> 38.3 mm, vias 0 -> 2
- net /SWDIO: track 14.3 -> 10.3 mm, vias 1 -> 0
- net /SWCLK: track 16.0 -> 12.2 mm, vias 1 -> 0
- net /NRST: track 15.8 -> 18.4 mm, vias 0 -> 2
- net /VBUS: track 7.69 -> 10.2 mm
- net /SELECT0: track 441.2 -> 442.9 mm, vias 16 -> 6
- net /SELECT1: track 446.3 -> 444.6 mm, vias 16 -> 6
- net /ADC1: track 57.0 -> 55.5 mm
- net /USB_D-: track 11.7 -> 10.3 mm
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- added copper zone on B.Cu, net +5V
Other:
- board text added: "Macrolev Rev 1.0 github.com/heiso/macrolev"
- board text removed: "Macrolev Rev 1.0"

Commit message: add caps on amux, change routing
Parts:
- added ! 8: SW_MX_Lekker_1u, Lekker switch:SW_MX_Lekker_1u, F.Cu at (216.2, 40.0)
- added " 3: SW_MX_Lekker_1u, Lekker switch:SW_MX_Lekker_1u, F.Cu at (121.0, 40.0)
- added $ * €: SW_MX_Lekker_1u, Lekker switch:SW_MX_Lekker_1u, F.Cu at (301.9, 59.0)
- added & 1: SW_MX_Lekker_1u, Lekker switch:SW_MX_Lekker_1u, F.Cu at (82.9, 40.0)
- added ' 4: SW_MX_Lekker_1u, Lekker switch:SW_MX_Lekker_1u, F.Cu at (140.0, 40.0)
- added ( 5: SW_MX_Lekker_1u, Lekker switch:SW_MX_Lekker_1u, F.Cu at (159.1, 40.0)
- added ) °: SW_MX_Lekker_1u, Lekker switch:SW_MX_Lekker_1u, F.Cu at (273.4, 40.0)
- added , ?: SW_MX_Lekker_1u, Lekker switch:SW_MX_Lekker_1u, F.Cu at (221.0, 97.2)
- added - _: SW_MX_Lekker_1u, Lekker switch:SW_MX_Lekker_1u, F.Cu at (292.4, 40.0)
- added : /: SW_MX_Lekker_1u, Lekker switch:SW_MX_Lekker_1u, F.Cu at (259.1, 97.2)
- added ; .: SW_MX_Lekker_1u, Lekker switch:SW_MX_Lekker_1u, F.Cu at (240.0, 97.2)
- added < >: SW_MX_Lekker_1u, Lekker switch:SW_MX_Lekker_1u, F.Cu at (87.6, 97.2)
- added = +: SW_MX_Lekker_1u, Lekker switch:SW_MX_Lekker_1u, F.Cu at (278.1, 97.2)
- added @ #: SW_MX_Lekker_1u, Lekker switch:SW_MX_Lekker_1u, F.Cu at (63.8, 40.0)
- added C14: 100n, Capacitor_SMD:C_0402_1005Metric_Pad0.74x0.62mm_HandSolder, B.Cu at (204.1, 63.5)
- added C15: 100n, Capacitor_SMD:C_0402_1005Metric_Pad0.74x0.62mm_HandSolder, B.Cu at (275.0, 64.5)
- added C16: 100n, Capacitor_SMD:C_0402_1005Metric_Pad0.74x0.62mm_HandSolder, B.Cu at (308.8, 66.5)
- added C17: 100n, Capacitor_SMD:C_0402_1005Metric_Pad0.74x0.62mm_HandSolder, B.Cu at (79.1, 64.2)
- added C18: 100n, Capacitor_SMD:C_0402_1005Metric_Pad0.74x0.62mm_HandSolder, B.Cu at (141.5, 64.6)
- added REF**: MountingHole_3mm_Pad_TopOnly, MountingHole:MountingHole_3mm_Pad_TopOnly, B.Cu at (291.2, 93.1)
- added REF**: MountingHole_3mm_Pad_TopOnly, MountingHole:MountingHole_3mm_Pad_TopOnly, B.Cu at (84.0, 82.1)
- added REF**: MountingHole_3mm_Pad_TopOnly, MountingHole:MountingHole_3mm_Pad_TopOnly, B.Cu at (180.4, 111.2)
- added ^ ¨: SW_MX_Lekker_1u, Lekker switch:SW_MX_Lekker_1u, F.Cu at (282.9, 59.0)
- added ` £: SW_MX_Lekker_1u, Lekker switch:SW_MX_Lekker_1u, F.Cu at (306.7, 78.1)
- added a: SW_MX_Lekker_1u, Lekker switch:SW_MX_Lekker_1u, F.Cu at (92.4, 59.0)
- added b: SW_MX_Lekker_1u, Lekker switch:SW_MX_Lekker_1u, F.Cu at (182.9, 97.2)
- added backspace: SW_MX_Lekker, Lekker switch:SW_MX_Lekker, F.Cu at (321.0, 40.0)
- added c: SW_MX_Lekker_1u, Lekker switch:SW_MX_Lekker_1u, F.Cu at (144.8, 97.2)
- added caps lock: SW_MX_Lekker_1.75u, Lekker switch:SW_MX_Lekker_1.75u, F.Cu at (71.0, 78.1)
- added cmd: SW_MX_Lekker_1.25u, Lekker switch:SW_MX_Lekker_1.25u, F.Cu at (123.3, 116.2)
- added cmd: SW_MX_Lekker_1.25u, Lekker switch:SW_MX_Lekker_1.25u, F.Cu at (242.4, 116.2)
- added ctrl: SW_MX_Lekker_1.75u, Lekker switch:SW_MX_Lekker_1.75u, F.Cu at (71.0, 116.2)
- added d: SW_MX_Lekker_1u, Lekker switch:SW_MX_Lekker_1u, F.Cu at (135.2, 78.1)
- added down: SW_MX_Lekker_1u, Lekker switch:SW_MX_Lekker_1u, F.Cu at (311.5, 116.2)
- added e: SW_MX_Lekker_1u, Lekker switch:SW_MX_Lekker_1u, F.Cu at (130.5, 59.0)
- added enter: SW_MX_Lekker, Lekker switch:SW_MX_Lekker, F.Cu at (328.1, 68.6)
- added esc: SW_MX_Lekker_1u, Lekker switch:SW_MX_Lekker_1u, F.Cu at (40.0, 40.0)
- added f: SW_MX_Lekker_1u, Lekker switch:SW_MX_Lekker_1u, F.Cu at (154.3, 78.1)
- added fn: SW_MX_Lekker_1u, Lekker switch:SW_MX_Lekker_1u, F.Cu at (40.0, 78.1)
- added fn2: SW_MX_Lekker_1u, Lekker switch:SW_MX_Lekker_1u, F.Cu at (40.0, 59.0)
- added g: SW_MX_Lekker_1u, Lekker switch:SW_MX_Lekker_1u, F.Cu at (173.3, 78.1)
- added h: SW_MX_Lekker_1u, Lekker switch:SW_MX_Lekker_1u, F.Cu at (192.4, 78.1)
- added i: SW_MX_Lekker_1u, Lekker switch:SW_MX_Lekker_1u, F.Cu at (225.7, 59.0)
- added j: SW_MX_Lekker_1u, Lekker switch:SW_MX_Lekker_1u, F.Cu at (211.4, 78.1)
- added k: SW_MX_Lekker_1u, Lekker switch:SW_MX_Lekker_1u, F.Cu at (230.5, 78.1)
- added l: SW_MX_Lekker_1u, Lekker switch:SW_MX_Lekker_1u, F.Cu at (249.6, 78.1)
- added left: SW_MX_Lekker_1u, Lekker switch:SW_MX_Lekker_1u, F.Cu at (292.4, 116.2)
- added lshift: SW_MX_Lekker_1.25u, Lekker switch:SW_MX_Lekker_1.25u, F.Cu at (66.2, 97.2)
- added lspace: SW_MX_Lekker, Lekker switch:SW_MX_Lekker, F.Cu at (156.7, 116.2)
- added m: SW_MX_Lekker_1u, Lekker switch:SW_MX_Lekker_1u, F.Cu at (268.6, 78.1)
- added n: SW_MX_Lekker_1u, Lekker switch:SW_MX_Lekker_1u, F.Cu at (201.9, 97.2)
- added o: SW_MX_Lekker_1u, Lekker switch:SW_MX_Lekker_1u, F.Cu at (244.8, 59.0)
- added option: SW_MX_Lekker_1.25u, Lekker switch:SW_MX_Lekker_1.25u, F.Cu at (99.5, 116.2)
- added option: SW_MX_Lekker_1u, Lekker switch:SW_MX_Lekker_1u, F.Cu at (263.8, 116.2)
- added p: SW_MX_Lekker_1u, Lekker switch:SW_MX_Lekker_1u, F.Cu at (263.8, 59.0)
- added q: SW_MX_Lekker_1u, Lekker switch:SW_MX_Lekker_1u, F.Cu at (97.2, 78.1)
- added r: SW_MX_Lekker_1u, Lekker switch:SW_MX_Lekker_1u, F.Cu at (149.5, 59.0)
- added right: SW_MX_Lekker_1u, Lekker switch:SW_MX_Lekker_1u, F.Cu at (330.5, 116.2)
- added rshift: SW_MX_Lekker, Lekker switch:SW_MX_Lekker, F.Cu at (313.8, 97.2)
- added rspace: SW_MX_Lekker, Lekker switch:SW_MX_Lekker, F.Cu at (204.3, 116.2)
- added s: SW_MX_Lekker_1u, Lekker switch:SW_MX_Lekker_1u, F.Cu at (116.2, 78.1)
- added t: SW_MX_Lekker_1u, Lekker switch:SW_MX_Lekker_1u, F.Cu at (168.6, 59.0)
- added tab: SW_MX_Lekker_1.5u, Lekker switch:SW_MX_Lekker_1.5u, F.Cu at (68.6, 59.0)
- added u: SW_MX_Lekker_1u, Lekker switch:SW_MX_Lekker_1u, F.Cu at (206.7, 59.0)
- added v: SW_MX_Lekker_1u, Lekker switch:SW_MX_Lekker_1u, F.Cu at (163.8, 97.2)
- added w: SW_MX_Lekker_1u, Lekker switch:SW_MX_Lekker_1u, F.Cu at (106.7, 97.2)
- added x: SW_MX_Lekker_1u, Lekker switch:SW_MX_Lekker_1u, F.Cu at (125.7, 97.2)
- added y: SW_MX_Lekker_1u, Lekker switch:SW_MX_Lekker_1u, F.Cu at (187.6, 59.0)
- added z: SW_MX_Lekker_1u, Lekker switch:SW_MX_Lekker_1u, F.Cu at (111.4, 59.0)
- added § 6: SW_MX_Lekker_1u, Lekker switch:SW_MX_Lekker_1u, F.Cu at (178.1, 40.0)
- added à 0: SW_MX_Lekker_1u, Lekker switch:SW_MX_Lekker_1u, F.Cu at (254.3, 40.0)
- added ç 9: SW_MX_Lekker_1u, Lekker switch:SW_MX_Lekker_1u, F.Cu at (235.3, 40.0)
- added è 7: SW_MX_Lekker_1u, Lekker switch:SW_MX_Lekker_1u, F.Cu at (197.2, 40.0)
- added é 2: SW_MX_Lekker_1u, Lekker switch:SW_MX_Lekker_1u, F.Cu at (101.9, 40.0)
- added ù %: SW_MX_Lekker_1u, Lekker switch:SW_MX_Lekker_1u, F.Cu at (287.6, 78.1)
- U1, U10, U11, U12, U13, U14, U16, U18, U19, U2, U20, U21, U22, U23, U24, U25, U26, U27, U28, U29, U3, U31, U33, U34, U35, U36, U37, U38, U39, U4, U40, U41, U42, U43, U44, U46, U47, U48, U49, U5, U50, U51, U52, U53, U54, U55, U56, U6, U64, U65, U66, U67, U7, U8, U9: footprint Lekker switch:SW_MX_Lekker_1u -> Package_TO_SOT_SMD:SOT-23; moved to B.Cu
- U15, U30, U57, U61, U62: footprint Lekker switch:SW_MX_Lekker -> Package_TO_SOT_SMD:SOT-23; moved to B.Cu
- U17: footprint Lekker switch:SW_MX_Lekker_1.5u -> Package_TO_SOT_SMD:SOT-23; moved to B.Cu
- U32, U58: footprint Lekker switch:SW_MX_Lekker_1.75u -> Package_TO_SOT_SMD:SOT-23; moved to B.Cu
- U45, U59, U60, U63: footprint Lekker switch:SW_MX_Lekker_1.25u -> Package_TO_SOT_SMD:SOT-23; moved to B.Cu
- moved R5 1.17 mm to (194.1, 47.0), turned to 90 degrees
- turned U1 to -45 degrees
- turned U10 to -45 degrees
- turned U11 to -45 degrees
- turned U12 to -45 degrees
- turned U13 to -45 degrees
- turned U14 to -45 degrees
- turned U15 to -45 degrees
- turned U16 to -45 degrees
- turned U17 to -45 degrees
- turned U18 to -45 degrees
- turned U19 to -45 degrees
- turned U2 to -45 degrees
- turned U20 to -45 degrees
- turned U21 to -45 degrees
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Routing:
- net +3.3VA: track 2049.5 -> 2058.1 mm
- net GND: track 38.5 -> 42.9 mm, vias 463 -> 541
- net /AMUX3:8: track 38.3 -> 34.4 mm
- net /AMUX0:13: track 33.4 -> 36.7 mm
- net /SELECT2: track 442.1 -> 444.8 mm
- net /AMUX2:9: track 32.0 -> 33.6 mm
- net /ADC0: track 113.8 -> 114.7 mm
- net /AMUX4:1: track 11.4 -> 12.1 mm
Other:
- board text added: "Macrolev Rev 1.0 github.com/heiso/macrolev Layout Mac ISO azerty (fr)"
- board text removed: "Macrolev Rev 1.0 github.com/heiso/macrolev"
