File: kicad/macrolev.kicad_pcb (KiCad board)
At the start: 2 copper layers, 309.6 x 95.2 mm, 184 parts, among them J1 USBC, J2 I2C, J3 DEBUG, SW1 RST_BTN, SW2 BOOT_BTN, U1 A1101ELHL, U10 A1101ELHL, U11 A1101ELHL, U12 A1101ELHL, U13 A1101ELHL, U14 A1101ELHL, U15 A1101ELHL, U16 A1101ELHL, U17 A1101ELHL, U18 A1101ELHL, U19 A1101ELHL, U2 A1101ELHL, U20 A1101ELHL, U21 A1101ELHL, U22 A1101ELHL, U23 A1101ELHL, U24 A1101ELHL, U25 A1101ELHL, U26 A1101ELHL, U27 A1101ELHL, U28 A1101ELHL, U29 A1101ELHL, U3 A1101ELHL, U30 A1101ELHL, U31 A1101ELHL, U32 A1101ELHL, U33 A1101ELHL, U34 A1101ELHL, U35 A1101ELHL, U36 A1101ELHL, U37 A1101ELHL, U38 A1101ELHL, U39 A1101ELHL, U4 A1101ELHL, U40 A1101ELHL, U41 A1101ELHL, U42 A1101ELHL, U43 A1101ELHL, U44 A1101ELHL, U45 A1101ELHL, U46 A1101ELHL, U47 A1101ELHL, U48 A1101ELHL, U49 A1101ELHL, U5 A1101ELHL, U50 A1101ELHL, U51 A1101ELHL, U52 A1101ELHL, U53 A1101ELHL, U54 A1101ELHL, U55 A1101ELHL, U56 A1101ELHL, U57 A1101ELHL, U58 A1101ELHL, U59 A1101ELHL, U6 A1101ELHL, U60 A1101ELHL, U61 A1101ELHL, U62 A1101ELHL, U63 A1101ELHL, U64 A1101ELHL, U65 A1101ELHL, U66 A1101ELHL, U67 A1101ELHL, U68 AMS1117-3.3, U69 STM32F411CEU6, U7 A1101ELHL, U8 A1101ELHL, U9 A1101ELHL, Y1 25MHz/20ppm/15pF

Commit message: wip: fix pcb
Parts:
- removed SW1: RST_BTN, switch:SKRPACE010
- removed SW2: BOOT_BTN, switch:SKRPACE010
- moved R4 9.51 mm to (171.9, 53.7), turned to 90 degrees
- turned enter to 90 degrees
Routing:
- net +3.3V: track 112.1 -> 84.0 mm
- net /BOOT0: track 22.3 -> 5.14 mm
- net /NRST: track 18.4 -> 10.8 mm, vias 2 -> 0
Other:
- outline, holes or cut-outs redrawn

Commit message: wip rev 1.1
Parts:
- removed J1: USBC, Connector_PinHeader_2.54mm:PinHeader_1x04_P2.54mm_Vertical
- removed R3: 10k, Resistor_SMD:R_0402_1005Metric_Pad0.72x0.64mm_HandSolder
- removed the REF** at (291.2, 93.1)
- removed the REF** at (84.0, 82.1)
- removed the REF** at (180.4, 111.2)
- added C10: 22u, Capacitor_SMD:C_0805_2012Metric_Pad1.18x1.45mm_HandSolder, B.Cu at (64.0, 32.2)
- added C11: 22u, Capacitor_SMD:C_0805_2012Metric_Pad1.18x1.45mm_HandSolder, B.Cu at (70.4, 36.2)
- added FB2: 120R, Inductor_SMD:L_0603_1608Metric_Pad1.05x0.95mm_HandSolder, B.Cu at (64.1, 34.2)
- added R6: 5.1K, Resistor_SMD:R_0402_1005Metric_Pad0.72x0.64mm_HandSolder, B.Cu at (49.3, 41.3)
- added R7: 5.1K, Resistor_SMD:R_0402_1005Metric_Pad0.72x0.64mm_HandSolder, B.Cu at (54.4, 41.3)
- added U68: AMS1117-3.3, Package_TO_SOT_SMD:SOT-223-3_TabPin2, B.Cu at (75.8, 35.0)
- added U70: GT-USB-7010ASV, JLCPCB:USB-C-SMD_G-SWITCH_GT-USB-7010ASV, B.Cu at (51.8, 33.5)
- J3: footprint Connector_PinHeader_2.54mm:PinHeader_1x04_P2.54mm_Vertical -> Connector_PinHeader_2.54mm:PinHeader_1x04_P2.54mm_Horizontal
- moved FID2 35.5 mm to (52.2, 78.4)
- moved J2 6.06 mm to (179.6, 68.9)
- moved C16 2.44 mm to (310.9, 65.3)
Routing:
- net +3.3VA: track 2058.1 -> 19.6 mm, vias 26 -> 0
- net /SELECT3: track 446.8 -> 4.11 mm, vias 8 -> 0
- net /SELECT0: track 442.9 -> 1.22 mm, vias 6 -> 0
- net /SELECT2: track 444.8 -> 3.90 mm, vias 8 -> 0
- net /SELECT1: track 444.6 -> 3.69 mm, vias 6 -> 0
- net /USB_D-: track 10.3 -> 0.00 mm
- net /USB_D+: track 10.2 -> 0.00 mm
- net /NRST: track 10.8 -> 2.53 mm
- net /AMUX0:10: track 51.0 -> 58.4 mm
- net +3.3V: track 84.0 -> 76.8 mm
- net /I2C_SCL: track 26.1 -> 20.2 mm
- net /VBUS: track 10.2 -> 4.95 mm
- net /I2C_SDA: track 28.2 -> 23.4 mm
- net /AMUX0:8: track 36.0 -> 38.2 mm
- net /AMUX3:8: vias 2 -> 0
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Other:
- copper layers 2 -> 4
- board text added: "Macrolev Rev 1.1 github.com/heiso/macrolev Layout Mac ISO azerty (fr)"
- board text removed: "Macrolev Rev 1.0 github.com/heiso/macrolev Layout Mac ISO azerty (fr)"
