File: kicad/macrolev.kicad_sch (KiCad schematic)
At the start: 182 parts, among them SW1 RotaryEncoder_Switch, U1 DRV2605LDGS, U10 GH39FKSW, U11 GH39FKSW, U12 GH39FKSW, U13 GH39FKSW, U14 GH39FKSW, U15 GH39FKSW, U16 GH39FKSW, U17 GH39FKSW, U18 GH39FKSW, U19 GH39FKSW, U2 GH39FKSW, U20 GH39FKSW, U21 GH39FKSW, U22 GH39FKSW, U23 GH39FKSW, U24 GH39FKSW, U25 GH39FKSW, U26 GH39FKSW, U27 GH39FKSW, U28 GH39FKSW, U29 GH39FKSW, U3 GH39FKSW, U30 GH39FKSW, U31 GH39FKSW, U32 GH39FKSW, U33 GH39FKSW, U34 GH39FKSW, U35 GH39FKSW, U36 GH39FKSW, U37 GH39FKSW, U38 GH39FKSW, U39 GH39FKSW, U4 GH39FKSW, U40 GH39FKSW, U41 GH39FKSW, U42 GH39FKSW, U43 GH39FKSW, U44 GH39FKSW, U45 GH39FKSW, U46 GH39FKSW, U47 GH39FKSW, U48 GH39FKSW, U49 GH39FKSW, U5 GH39FKSW, U50 GH39FKSW, U51 GH39FKSW, U52 GH39FKSW, U53 GH39FKSW, U54 GH39FKSW, U55 GH39FKSW, U56 GH39FKSW, U57 GH39FKSW, U58 GH39FKSW, U59 GH39FKSW, U6 GH39FKSW, U60 GH39FKSW, U61 GH39FKSW, U62 GH39FKSW, U63 GH39FKSW, U64 GH39FKSW, U65 GH39FKSW, U7 GH39FKSW, U8 GH39FKSW, U9 GH39FKSW, X1 12MHz

Commit message: 📝  Add wooting 60HE pictures
Parts:
- removed C4, C5: 1uF, Capacitor_SMD:C_0402_1005Metric, symbol Device:C
- removed R2, R3: 10K, Resistor_SMD:R_0402_1005Metric, symbol Device:R
- removed TP1: In/Trig, TestPoint:TestPoint_Pad_D1.5mm, symbol Connector:TestPoint
- removed TP2: +, TestPoint:TestPoint_Pad_D1.5mm, symbol Connector:TestPoint
- removed TP3: -, TestPoint:TestPoint_Pad_1.5x1.5mm, symbol Connector:TestPoint
- removed U1: DRV2605LDGS, Package_SO:VSSOP-10_3x3mm_P0.5mm, symbol Driver_Haptic:DRV2605LDGS
- added I2C1: Conn_01x02, symbol Connector_Generic:Conn_01x02
- renumbered C12 to C10, C13 to C11, C14 to C12, C15 to C13, C16 to C14, C17 to C15, C18 to C16, C19 to C17, C20 to C18, C21 to C19, C6 to C4, C7 to C5, C8 to C6, C9 to C7, C10 to C8, C11 to C9, R4 to R2, R5 to R3, R6 to R4, R7 to R5, R11 to R6, R8 to R7, R9 to R8, R10 to R9, U2 to U1, U11 to U10, U12 to U11, U13 to U12, U14 to U13, U15 to U14, U16 to U15, U17 to U16, U18 to U17, U19 to U18, U20 to U19, U3 to U2, U21 to U20, U22 to U21, U23 to U22, U24 to U23, U25 to U24, U26 to U25, U27 to U26, U28 to U27, U29 to U28, U30 to U29, U4 to U3, U31 to U30, U32 to U31, U33 to U32, U34 to U33, U35 to U34, U36 to U35, U37 to U36, U38 to U37, U39 to U38, U40 to U39, U5 to U4, U41 to U40, U42 to U41, U43 to U42, U44 to U43, U45 to U44, U46 to U45, U47 to U46, U48 to U47, U49 to U48, U50 to U49, U6 to U5, U51 to U50, U52 to U51, U53 to U52, U54 to U53, U55 to U54, U56 to U55, U57 to U56, U58 to U57, U59 to U58, U60 to U59, U7 to U6, U61 to U60, U62 to U61, U63 to U62, U64 to U63, U65 to U64, U8 to U7, U9 to U8, U10 to U9
Connections:
- net SCL0: now also I2C1.2 (Pin_2)
- net SDA0: now also I2C1.1 (Pin_1)
- net VBUS: now also MCU1.13 (GPIO10)
Other:
- note added: "CHOOSE CONNECTOR FOR I2C"
- note added: "TODO"
- note removed: "HAPTIC DRIVER"
- moved on the sheet: BOOT1, C7, Flash1, R2, R3

Commit message: pcb rev1.0
Parts:
- removed AM0:1: ESC, void_switch:VoidSwitch_1u_SMD, symbol voidswitch:VoidSwitch
- removed AM0:10: Z, void_switch:VoidSwitch_1u_SMD, symbol voidswitch:VoidSwitch
- removed AM0:11: 2, void_switch:VoidSwitch_1u_SMD, symbol voidswitch:VoidSwitch
- removed AM0:12: W, void_switch:VoidSwitch_1u_SMD, symbol voidswitch:VoidSwitch
- removed AM0:13: LAlt, void_switch:VoidSwitch_1.25u_SMD, symbol voidswitch:VoidSwitch
- removed AM0:14: S, void_switch:VoidSwitch_1u_SMD, symbol voidswitch:VoidSwitch
- removed AM0:15: 3, void_switch:VoidSwitch_1u_SMD, symbol voidswitch:VoidSwitch
- removed AM0:16: E, void_switch:VoidSwitch_1u_SMD, symbol voidswitch:VoidSwitch
- removed AM0:2: Tab, void_switch:VoidSwitch_1.5u_SMD, symbol voidswitch:VoidSwitch
- removed AM0:3: CAPS, void_switch:VoidSwitch_1.75u_SMD, symbol voidswitch:VoidSwitch
- removed AM0:4: LShift, void_switch:VoidSwitch_1.25u_SMD, symbol voidswitch:VoidSwitch
- removed AM0:5: LCtrl, void_switch:VoidSwitch_1.25u_SMD, symbol voidswitch:VoidSwitch
- removed AM0:6: 1, void_switch:VoidSwitch_1u_SMD, symbol voidswitch:VoidSwitch
- removed AM0:7: Super, void_switch:VoidSwitch_1.25u_SMD, symbol voidswitch:VoidSwitch
- removed AM0:8: Q, void_switch:VoidSwitch_1u_SMD, symbol voidswitch:VoidSwitch
- removed AM0:9: A, void_switch:VoidSwitch_1u_SMD, symbol voidswitch:VoidSwitch
- removed AM1:1: X, void_switch:VoidSwitch_1u_SMD, symbol voidswitch:VoidSwitch
- removed AM1:10: T, void_switch:VoidSwitch_1u_SMD, symbol voidswitch:VoidSwitch
- removed AM1:11: G, void_switch:VoidSwitch_1u_SMD, symbol voidswitch:VoidSwitch
- removed AM1:12: B, void_switch:VoidSwitch_1u_SMD, symbol voidswitch:VoidSwitch
- removed AM1:13: 6, void_switch:VoidSwitch_1u_SMD, symbol voidswitch:VoidSwitch
- removed AM1:14: Y, void_switch:VoidSwitch_1u_SMD, symbol voidswitch:VoidSwitch
- removed AM1:15: H, void_switch:VoidSwitch_1u_SMD, symbol voidswitch:VoidSwitch
- removed AM1:2: D, void_switch:VoidSwitch_1u_SMD, symbol voidswitch:VoidSwitch
- removed AM1:3: C, void_switch:VoidSwitch_1u_SMD, symbol voidswitch:VoidSwitch
- removed AM1:4: 4, void_switch:VoidSwitch_1u_SMD, symbol voidswitch:VoidSwitch
- removed AM1:5: R, void_switch:VoidSwitch_1u_SMD, symbol voidswitch:VoidSwitch
- removed AM1:6: F, void_switch:VoidSwitch_1u_SMD, symbol voidswitch:VoidSwitch
- removed AM1:7: V, void_switch:VoidSwitch_1u_SMD, symbol voidswitch:VoidSwitch
- removed AM1:8: LSpace, void_switch:VoidSwitch_1.75u_SMD, symbol voidswitch:VoidSwitch
- removed AM1:9: 5, void_switch:VoidSwitch_1u_SMD, symbol voidswitch:VoidSwitch
- removed AM2:1: RSpace, void_switch:VoidSwitch_1.75u_SMD, symbol voidswitch:VoidSwitch
- removed AM2:10: Comma, void_switch:VoidSwitch_1u_SMD, symbol voidswitch:VoidSwitch
- removed AM2:11: 9, void_switch:VoidSwitch_1u_SMD, symbol voidswitch:VoidSwitch
- removed AM2:12: O, void_switch:VoidSwitch_1u_SMD, symbol voidswitch:VoidSwitch
- removed AM2:2: N, void_switch:VoidSwitch_1u_SMD, symbol voidswitch:VoidSwitch
- removed AM2:3: 7, void_switch:VoidSwitch_1u_SMD, symbol voidswitch:VoidSwitch
- removed AM2:4: U, void_switch:VoidSwitch_1u_SMD, symbol voidswitch:VoidSwitch
- removed AM2:5: J, void_switch:VoidSwitch_1u_SMD, symbol voidswitch:VoidSwitch
- removed AM2:6: M, void_switch:VoidSwitch_1u_SMD, symbol voidswitch:VoidSwitch
- removed AM2:7: 8, void_switch:VoidSwitch_1u_SMD, symbol voidswitch:VoidSwitch
- removed AM2:8: I, void_switch:VoidSwitch_1u_SMD, symbol voidswitch:VoidSwitch
- removed AM2:9: K, void_switch:VoidSwitch_1u_SMD, symbol voidswitch:VoidSwitch
- removed AM3:1: RAlt, void_switch:VoidSwitch_1.25u_SMD, symbol voidswitch:VoidSwitch
- removed AM3:10: LBrack, void_switch:VoidSwitch_1u_SMD, symbol voidswitch:VoidSwitch
- removed AM3:11: Quot, void_switch:VoidSwitch_1u_SMD, symbol voidswitch:VoidSwitch
- removed AM3:12: Equal, void_switch:VoidSwitch_1u_SMD, symbol voidswitch:VoidSwitch
- removed AM3:13: RBrack, void_switch:VoidSwitch_1u_SMD, symbol voidswitch:VoidSwitch
- removed AM3:2: L, void_switch:VoidSwitch_1u_SMD, symbol voidswitch:VoidSwitch
- removed AM3:3: Period, void_switch:VoidSwitch_1u_SMD, symbol voidswitch:VoidSwitch
- removed AM3:4: Zero, void_switch:VoidSwitch_1u_SMD, symbol voidswitch:VoidSwitch
- removed AM3:5: Fn, void_switch:VoidSwitch_1.25u_SMD, symbol voidswitch:VoidSwitch
- removed AM3:6: P, void_switch:VoidSwitch_1u_SMD, symbol voidswitch:VoidSwitch
- removed AM3:7: Semi, void_switch:VoidSwitch_1u_SMD, symbol voidswitch:VoidSwitch
- removed AM3:8: Slash, void_switch:VoidSwitch_1u_SMD, symbol voidswitch:VoidSwitch
- removed AM3:9: Minus, void_switch:VoidSwitch_1u_SMD, symbol voidswitch:VoidSwitch
- removed AM4:1: RShift, void_switch:VoidSwitch_1.5u_SMD, symbol voidswitch:VoidSwitch
- removed AM4:2: LEFT, void_switch:VoidSwitch_1u_SMD, symbol voidswitch:VoidSwitch
- removed AM4:3: Enter, void_switch:VoidSwitch_1.75u_SMD, symbol voidswitch:VoidSwitch
- removed AM4:4: BS, void_switch:VoidSwitch_1.5u_SMD, symbol voidswitch:VoidSwitch
- removed AM4:5: Bslash, void_switch:VoidSwitch_1u_SMD, symbol voidswitch:VoidSwitch
- removed AM4:6: UP, void_switch:VoidSwitch_1u_SMD, symbol voidswitch:VoidSwitch
- removed AM4:7: DOWN, void_switch:VoidSwitch_1u_SMD, symbol voidswitch:VoidSwitch
- removed AM4:8: RIGHT, void_switch:VoidSwitch_1u_SMD, symbol voidswitch:VoidSwitch
- removed BOOT1, RST1: TS-1187A-B-A-B, footprint:SW-SMD_4P-L5.1-W5.1-P3.70-LS6.5-TL-2, symbol default_lib:TS-1187A-B-A-B
- removed C14, C15: 100nF, Capacitor_SMD:C_0402_1005Metric, symbol Device:C
- removed C16, C17: 10uF, Capacitor_SMD:C_0402_1005Metric, symbol Device:C
- removed C18, C19: 22pF, Capacitor_SMD:C_0402_1005Metric, symbol Device:C
- removed Debug1, UART1: Conn_01x05, Connector_PinHeader_2.54mm:PinHeader_1x05_P2.54mm_Vertical, symbol Connector_Generic:Conn_01x05
- removed Flash1: W25Q128JVS, Package_SO:SOIC-8_5.23x5.23mm_P1.27mm, symbol Memory_Flash:W25Q128JVS
- removed I2C1: Conn_01x02, symbol Connector_Generic:Conn_01x02
- removed LDO1, LDO2: NCP1117-3.3_SOT223, Package_TO_SOT_SMD:SOT-223-3_TabPin2, symbol Regulator_Linear:NCP1117-3.3_SOT223
- removed MCU1: RP2040, footprint:LQFN-56_L7.0-W7.0-P0.4-EP, symbol default_lib:RP2040
- removed R1, R7, R8, R9: 10k, Resistor_SMD:R_0402_1005Metric, symbol Device:R
- removed R2, R6: 1k, Resistor_SMD:R_0402_1005Metric, symbol Device:R
- removed SW1: RotaryEncoder_Switch, Rotary_Encoder:RotaryEncoder_Alps_EC11E-Switch_Vertical_H20mm, symbol Device:RotaryEncoder_Switch
- removed U1, U10, U11, U12, U13, U14, U15, U16, U17, U18, U19, U2, U20, U21, U22, U23, U24, U25, U26, U27, U28, U29, U3, U30, U31, U32, U33, U34, U35, U36, U37, U38, U39, U4, U40, U41, U42, U43, U44, U45, U46, U47, U48, U49, U5, U50, U51, U52, U53, U54, U55, U56, U57, U58, U59, U6, U60, U61, U62, U63, U64, U7, U8, U9: GH39FKSW, Package_TO_SOT_SMD:SOT-23, symbol 49e:Hall_Sensor
- removed USB1: Conn_01x04, Connector_PinHeader_2.54mm:PinHeader_1x04_P2.54mm_Vertical, symbol Connector_Generic:Conn_01x04
- removed X1: 12MHz, footprint:OSC-SMD_4P-L3.2-W2.5-BL, symbol default_lib:X322512MSB4SI
- added AMUX0: CD74HC4067SM, Package_SO:SSOP-24_5.3x8.2mm_P0.65mm, symbol 74xx:CD74HC4067SM
- added D1: RED, LED_SMD:LED_0603_1608Metric_Pad1.05x0.95mm_HandSolder, symbol Device:LED
- added FB1, FB2: 120R, Inductor_SMD:L_0603_1608Metric_Pad1.05x0.95mm_HandSolder, symbol Device:FerriteBead
- added J2: I2C, Connector_PinHeader_2.54mm:PinHeader_1x04_P2.54mm_Vertical, symbol Connector:Conn_01x04_Pin
- added J3: DEBUG, Connector_PinHeader_2.54mm:PinHeader_1x04_P2.54mm_Vertical, symbol Connector:Conn_01x04_Pin
- added J4: USBC, Connector_PinHeader_2.54mm:PinHeader_1x04_P2.54mm_Vertical, symbol Connector:Conn_01x04_Pin
- added SW1: BOOT_BTN, switch:SKRPACE010, symbol Switch:SW_Push_Dual
- added SW2: RST_BTN, switch:SKRPACE010, symbol Switch:SW_Push_Dual
- added U1, U10, U11, U12, U13, U14, U16, U18, U19, U2, U20, U21, U22, U23, U24, U25, U26, U27, U28, U29, U3, U31, U33, U34, U35, U36, U37, U38, U39, U4, U40, U41, U42, U43, U44, U46, U47, U48, U49, U5, U50, U51, U52, U53, U54, U55, U56, U6, U64, U65, U66, U67, U7, U8, U9: A1101ELHL, Lekker switch:SW_MX_Lekker_1u, symbol Sensor_Magnetic:A1101ELHL
- added U15, U30, U57, U61, U62: A1101ELHL, Lekker switch:SW_MX_Lekker, symbol Sensor_Magnetic:A1101ELHL
- added U17: A1101ELHL, Lekker switch:SW_MX_Lekker_1.5u, symbol Sensor_Magnetic:A1101ELHL
- added U32, U58: A1101ELHL, Lekker switch:SW_MX_Lekker_1.75u, symbol Sensor_Magnetic:A1101ELHL
- added U45, U59, U60, U63: A1101ELHL, Lekker switch:SW_MX_Lekker_1.25u, symbol Sensor_Magnetic:A1101ELHL
- added U68: AMS1117-3.3, Package_TO_SOT_SMD:SOT-223-3_TabPin2, symbol Regulator_Linear:AMS1117-3.3
- added U69: STM32F411CEU6, Package_DFN_QFN:QFN-48-1EP_7x7mm_P0.5mm_EP5.6x5.6mm, symbol MCU_ST_STM32F4:STM32F411CEUx
- added Y1: 25MHz/20ppm/15pF, Crystal:Crystal_SMD_3225-4Pin_3.2x2.5mm_HandSoldering, symbol Device:Crystal_GND24
- C1: value 100nF -> 10u; footprint Capacitor_SMD:C_0402_1005Metric -> Capacitor_SMD:C_0603_1608Metric_Pad1.08x0.95mm_HandSolder; LCSC C1525 -> (none)
- C10: value 100nF -> 22u; footprint Capacitor_SMD:C_0402_1005Metric -> Capacitor_SMD:C_0805_2012Metric_Pad1.18x1.45mm_HandSolder; LCSC C1525 -> (none)
- C11: value 10uF -> 22u; footprint Capacitor_SMD:C_0402_1005Metric -> Capacitor_SMD:C_0805_2012Metric_Pad1.18x1.45mm_HandSolder; LCSC C15525 -> (none)
- C12, C13: value 100nF -> 20p; footprint Capacitor_SMD:C_0402_1005Metric -> Capacitor_SMD:C_0402_1005Metric_Pad0.74x0.62mm_HandSolder; LCSC C1525 -> (none)
- C2, C3, C4: value 100nF -> 100n; footprint Capacitor_SMD:C_0402_1005Metric -> Capacitor_SMD:C_0402_1005Metric_Pad0.74x0.62mm_HandSolder; LCSC C1525 -> (none)
- C5, C9: value 1uF -> 100n; footprint Capacitor_SMD:C_0402_1005Metric -> Capacitor_SMD:C_0402_1005Metric_Pad0.74x0.62mm_HandSolder; LCSC C52923 -> (none)
- C6: value 10uF -> 10n; footprint Capacitor_SMD:C_0402_1005Metric -> Capacitor_SMD:C_0402_1005Metric_Pad0.74x0.62mm_HandSolder; LCSC C15525 -> (none)
- C7, C8: value 100nF -> 1u; footprint Capacitor_SMD:C_0402_1005Metric -> Capacitor_SMD:C_0402_1005Metric_Pad0.74x0.62mm_HandSolder; LCSC C1525 -> (none)
- R3: footprint Resistor_SMD:R_0402_1005Metric -> Resistor_SMD:R_0402_1005Metric_Pad0.72x0.64mm_HandSolder; LCSC C25744 -> (none)
- R4: value 27 -> 10k; footprint Resistor_SMD:R_0402_1005Metric -> Resistor_SMD:R_0402_1005Metric_Pad0.72x0.64mm_HandSolder; LCSC C25100 -> (none)
- R5: value 27 -> 5.1k; footprint Resistor_SMD:R_0402_1005Metric -> Resistor_SMD:R_0402_1005Metric_Pad0.72x0.64mm_HandSolder; LCSC C25100 -> (none)
Connections:
- net +1V0 is gone; now on net +3.3V: C1.1, C2.1, C5.1
- net D- is gone; now on net GND: R5.2
- net QSPI_SS is gone; now on net +3.3V: R3.1
- net +3.3V: now also D1.2 (A), FB1.2, J2.4 (Pin_4), J3.4 (Pin_4), SW2.2, SW2.4, U68.2 (VO), U69.1 (VBAT), U69.24 (VDD), U69.36 (VDD), U69.48 (VDD); no longer C10.1, C12.1, C13.1, C7.1, C9.1, R3.2
- net +3.3VA: now also C6.1, C7.1, AMUX0.24 (VCC), FB1.1, U1.1 (VCC), U10.1 (VCC), U11.1 (VCC), U12.1 (VCC), U13.1 (VCC), U14.1 (VCC), U15.1 (VCC), U16.1 (VCC), U17.1 (VCC), U18.1 (VCC), U19.1 (VCC), U2.1 (VCC), U20.1 (VCC), U21.1 (VCC), U22.1 (VCC), U23.1 (VCC), U24.1 (VCC), U25.1 (VCC), U26.1 (VCC), U27.1 (VCC), U28.1 (VCC), U29.1 (VCC), U3.1 (VCC), U30.1 (VCC), U31.1 (VCC), U32.1 (VCC), U33.1 (VCC), U34.1 (VCC), U35.1 (VCC), U36.1 (VCC), U37.1 (VCC), U38.1 (VCC), U39.1 (VCC), U4.1 (VCC), U40.1 (VCC), U41.1 (VCC), U42.1 (VCC), U43.1 (VCC), U44.1 (VCC), U45.1 (VCC), U46.1 (VCC), U47.1 (VCC), U48.1 (VCC), U49.1 (VCC), U5.1 (VCC), U50.1 (VCC), U51.1 (VCC), U52.1 (VCC), U53.1 (VCC), U54.1 (VCC), U55.1 (VCC), U56.1 (VCC), U57.1 (VCC), U58.1 (VCC), U59.1 (VCC), U6.1 (VCC), U60.1 (VCC), U61.1 (VCC), U62.1 (VCC), U63.1 (VCC), U64.1 (VCC), U65.1 (VCC), U66.1 (VCC), U67.1 (VCC), U69.9 (VDDA), U7.1 (VCC), U8.1 (VCC), U9.1 (VCC)
- net ADC0: now also AMUX0.1 (COM), U69.13 (PA3); no longer AMUX1.1 (COM)
- net ADC1: now also AMUX1.1 (COM), U69.14 (PA4); no longer AMUX2.1 (COM)
- net ADC2: now also AMUX2.1 (COM), U69.15 (PA5); no longer AMUX3.1 (COM)
- net ADC3: now also AMUX3.1 (COM), U69.16 (PA6); no longer AMUX4.1 (COM)
- net AMUX0:0: now also AMUX0.9 (I0), U46.2 (VOUT); no longer AMUX1.9 (I0)
- net AMUX0:1: now also AMUX0.8 (I1), U59.2 (VOUT); no longer AMUX1.8 (I1)
- net AMUX0:10: now also AMUX0.21 (I10), U1.2 (VOUT); no longer AMUX1.21 (I10)
- net AMUX0:11: now also AMUX0.20 (I11), U16.2 (VOUT); no longer AMUX1.20 (I11)
- net AMUX0:12: now also AMUX0.19 (I12), U31.2 (VOUT); no longer AMUX1.19 (I12)
- net AMUX0:13: now also AMUX0.18 (I13), U45.2 (VOUT); no longer AMUX1.18 (I13)
- net AMUX0:14: now also AMUX0.17 (I14), U32.2 (VOUT); no longer AMUX1.17 (I14)
- net AMUX0:15: now also AMUX0.16 (I15), U58.2 (VOUT); no longer AMUX1.16 (I15)
- net AMUX0:2: now also AMUX0.7 (I2), U33.2 (VOUT); no longer AMUX1.7 (I2)
- net AMUX0:3: now also AMUX0.6 (I3), U47.2 (VOUT); no longer AMUX1.6 (I3)
- net AMUX0:4: now also AMUX0.5 (I4), U19.2 (VOUT); no longer AMUX1.5 (I4)
- net AMUX0:5: now also AMUX0.4 (I5), U4.2 (VOUT); no longer AMUX1.4 (I5)
- net AMUX0:6: now also AMUX0.3 (I6), U18.2 (VOUT); no longer AMUX1.3 (I6)
- net AMUX0:7: now also AMUX0.2 (I7), U3.2 (VOUT); no longer AMUX1.2 (I7)
- net AMUX0:8: now also AMUX0.23 (I8), U2.2 (VOUT); no longer AMUX1.23 (I8)
- net AMUX0:9: now also AMUX0.22 (I9), U17.2 (VOUT); no longer AMUX1.22 (I9)
- net AMUX1:0: now also AMUX1.9 (I0), U61.2 (VOUT); no longer AMUX2.9 (I0)
- net AMUX1:1: now also AMUX1.8 (I1), U36.2 (VOUT); no longer AMUX2.8 (I1)
- net AMUX1:10: now also AMUX1.21 (I10), U20.2 (VOUT); no longer AMUX2.21 (I10)
- net AMUX1:11: now also AMUX1.20 (I11), U34.2 (VOUT); no longer AMUX2.20 (I11)
- net AMUX1:12: now also AMUX1.19 (I12), U60.2 (VOUT); no longer AMUX2.19 (I12)
- net AMUX1:13: now also AMUX1.18 (I13), U48.2 (VOUT); no longer AMUX2.18 (I13)
- net AMUX1:14: now also AMUX1.17 (I14), U35.2 (VOUT); no longer AMUX2.17 (I14)
- net AMUX1:15: now also AMUX1.16 (I15), U49.2 (VOUT); no longer AMUX2.16 (I15)
- net AMUX1:2: now also AMUX1.7 (I2), U50.2 (VOUT); no longer AMUX2.7 (I2)
- net AMUX1:3: now also AMUX1.6 (I3), U51.2 (VOUT); no longer AMUX2.6 (I3)
- net AMUX1:4: now also AMUX1.5 (I4), U37.2 (VOUT); no longer AMUX2.5 (I4)
- net AMUX1:5: now also AMUX1.4 (I5), U22.2 (VOUT); no longer AMUX2.4 (I5)
- net AMUX1:6: now also AMUX1.3 (I6), U7.2 (VOUT); no longer AMUX2.3 (I6)
- net AMUX1:7: now also AMUX1.2 (I7), U21.2 (VOUT); no longer AMUX2.2 (I7)
- net AMUX1:8: now also AMUX1.23 (I8), U6.2 (VOUT); no longer AMUX2.23 (I8)
- net AMUX1:9: now also AMUX1.22 (I9), U5.2 (VOUT); no longer AMUX2.22 (I9)
- net AMUX2:0: now also AMUX2.9 (I0), U53.2 (VOUT); no longer AMUX3.9 (I0)
- net AMUX2:1: now also AMUX2.8 (I1), U63.2 (VOUT); no longer AMUX3.8 (I1)
- net AMUX2:10: now also AMUX2.21 (I10), U8.2 (VOUT); no longer AMUX3.21 (I10)
- net AMUX2:11: now also AMUX2.20 (I11), U23.2 (VOUT); no longer AMUX3.20 (I11)
- net AMUX2:12: now also AMUX2.19 (I12), U38.2 (VOUT); no longer AMUX3.19 (I12)
- net AMUX2:13: now also AMUX2.18 (I13), U62.2 (VOUT); no longer AMUX3.18 (I13)
- net AMUX2:14: now also AMUX2.17 (I14), U52.2 (VOUT); no longer AMUX3.17 (I14)
- net AMUX2:15: now also AMUX2.16 (I15), U39.2 (VOUT); no longer AMUX3.16 (I15)
- net AMUX2:2: now also AMUX2.7 (I2), U54.2 (VOUT); no longer AMUX3.7 (I2)
- net AMUX2:3: now also AMUX2.6 (I3), U40.2 (VOUT); no longer AMUX3.6 (I3)
- net AMUX2:4: now also AMUX2.5 (I4), U26.2 (VOUT); no longer AMUX3.5 (I4)
- net AMUX2:5: now also AMUX2.4 (I5), U25.2 (VOUT); no longer AMUX3.4 (I5)
- net AMUX2:6: now also AMUX2.3 (I6), U11.2 (VOUT); no longer AMUX3.3 (I6)
- net AMUX2:7: now also AMUX2.2 (I7), U10.2 (VOUT); no longer AMUX3.2 (I7)
- net AMUX2:8: now also AMUX2.23 (I8), U24.2 (VOUT); no longer AMUX3.23 (I8)
- net AMUX2:9: now also AMUX2.22 (I9), U9.2 (VOUT); no longer AMUX3.22 (I9)
- net AMUX3:0: now also AMUX3.9 (I0), U65.2 (VOUT); no longer AMUX4.9 (I0)
- net AMUX3:1: now also AMUX3.8 (I1), U43.2 (VOUT); no longer AMUX4.8 (I1)
- net AMUX3:10: now also AMUX3.21 (I10), U27.2 (VOUT); no longer AMUX4.21 (I10)
- net AMUX3:11: now also AMUX3.20 (I11), U41.2 (VOUT); no longer AMUX4.20 (I11)
- net AMUX3:12: now also AMUX3.19 (I12), U55.2 (VOUT); no longer AMUX4.19 (I12)
- net AMUX3:13: now also AMUX3.18 (I13), U64.2 (VOUT); no longer AMUX4.18 (I13)
- net AMUX3:14: now also AMUX3.17 (I14), U42.2 (VOUT); no longer AMUX4.17 (I14)
- net AMUX3:15: now also AMUX3.16 (I15), U56.2 (VOUT); no longer AMUX4.16 (I15)
- net AMUX3:2: now also AMUX3.7 (I2), U66.2 (VOUT); no longer AMUX4.7 (I2)
- net AMUX3:3: now also AMUX3.6 (I3), U57.2 (VOUT); no longer AMUX4.6 (I3)
- net AMUX3:4: now also AMUX3.5 (I4), U44.2 (VOUT); no longer AMUX4.5 (I4)
- net AMUX3:5: now also AMUX3.4 (I5), U29.2 (VOUT); no longer AMUX4.4 (I5)
- net AMUX3:6: now also AMUX3.3 (I6), U14.2 (VOUT); no longer AMUX4.3 (I6)
- net AMUX3:7: now also AMUX3.2 (I7), U28.2 (VOUT); no longer AMUX4.2 (I7)
- net AMUX3:8: now also AMUX3.23 (I8), U13.2 (VOUT); no longer AMUX4.23 (I8)
- net AMUX3:9: now also AMUX3.22 (I9), U12.2 (VOUT); no longer AMUX4.22 (I9)
- net GND: now also R4.1, AMUX0.12 (GND), AMUX0.15 (~{E}), J2.1 (Pin_1), J3.1 (Pin_1), J4.1 (Pin_1), SW1.2, SW1.4, U1.3 (GND), U10.3 (GND), U11.3 (GND), U12.3 (GND), U13.3 (GND), U14.3 (GND), U15.3 (GND), U16.3 (GND), U17.3 (GND), U18.3 (GND), U19.3 (GND), U2.3 (GND), U20.3 (GND), U21.3 (GND), U22.3 (GND), U23.3 (GND), U24.3 (GND), U25.3 (GND), U26.3 (GND), U27.3 (GND), U28.3 (GND), U29.3 (GND), U3.3 (GND), U30.3 (GND), U31.3 (GND), U32.3 (GND), U33.3 (GND), U34.3 (GND), U35.3 (GND), U36.3 (GND), U37.3 (GND), U38.3 (GND), U39.3 (GND), U4.3 (GND), U40.3 (GND), U41.3 (GND), U42.3 (GND), U43.3 (GND), U44.3 (GND), U45.3 (GND), U46.3 (GND), U47.3 (GND), U48.3 (GND), U49.3 (GND), U5.3 (GND), U50.3 (GND), U51.3 (GND), U52.3 (GND), U53.3 (GND), U54.3 (GND), U55.3 (GND), U56.3 (GND), U57.3 (GND), U58.3 (GND), U59.3 (GND), U6.3 (GND), U60.3 (GND), U61.3 (GND), U62.3 (GND), U63.3 (GND), U64.3 (GND), U65.3 (GND), U66.3 (GND), U67.3 (GND), U68.1 (GND), U69.23 (VSS), U69.35 (VSS), U69.47 (VSS), U69.49 (VSS), U69.8 (VSSA), U7.3 (GND), U8.3 (GND), U9.3 (GND), Y1.2, Y1.4
- net SELECT0: now also AMUX0.10 (S0), U69.25 (PB12)
- net SELECT1: now also AMUX0.11 (S1), U69.26 (PB13)
- net SELECT2: now also AMUX0.14 (S2), U69.27 (PB14)
- net SELECT3: now also AMUX0.13 (S3), U69.28 (PB15)
- net SWCLK: now also J3.2 (Pin_2), U69.37 (PA14)
- net VBUS: now also FB2.1, J4.2 (Pin_2); no longer C6.1
- net at R5.1: now also D1.1 (K)
- net D+ renamed BOOT0
- net BOOT0: now also SW2.1, SW2.3, U69.44 (BOOT0)
- new net +5V: C10.1, FB2.2, U68.3 (VI)
- new net ADC4: AMUX4.1 (COM), U69.17 (PA7)
- new net AMUX4:0: AMUX4.9 (I0), U67.2 (VOUT)
- new net AMUX4:1: AMUX4.8 (I1), U30.2 (VOUT)
- new net AMUX4:2: AMUX4.7 (I2), U15.2 (VOUT)
- new net HSE_IN: C12.1, U69.5 (PH0), Y1.1
- new net HSE_OUT: C13.1, U69.6 (PH1), Y1.3
- new net I2C_SCL: J2.3 (Pin_3), U69.42 (PB6)
- new net I2C_SDA: J2.2 (Pin_2), U69.43 (PB7)
- new net NRST: C9.1, R3.2, SW1.1, SW1.3, U69.7 (NRST)
- new net SWDIO: J3.3 (Pin_3), U69.34 (PA13)
- new net USB_D+: J4.4 (Pin_4), U69.33 (PA12)
- new net USB_D-: J4.3 (Pin_3), U69.32 (PA11)
- no-connect marks 1 -> 33
Other:
- note added: "Analog Multiplexer"
- note added: "Buttons"
- note added: "C = (15pF - 5pF)*2 = 20pF"
- note added: "Connectors"
- note added: "Crystal"
- note added: "Power"
- note removed: "CHOOSE CONNECTOR FOR I2C"
- note removed: "Close to rp2040 pins 46-47"
- note removed: "DECOUPLING CAPACITORS (Close to pins)"
- note removed: "FLASH"
- note removed: "OSCILLATOR"
- note removed: "POWER"
- note removed: "ROTARY ENCODER"
- note removed: "TODO"
- note removed: "USB"
- note removed: "the performance of the ADC will be compromised at voltages below 2.97V"
- note removed: "this particular flash device appears to not need external pull-up, solder jumper just in case"
- company: (none) -> Heiso
- title: (none) -> Macrolev
