File: kicad_2/kicad_2.kicad_pcb (KiCad board)
At the start: 2 copper layers, 309.6 x 95.2 mm, 73 parts, among them U1 A1101ELHL, U10 A1101ELHL, U11 A1101ELHL, U12 A1101ELHL, U13 A1101ELHL, U14 A1101ELHL, U15 A1101ELHL, U16 A1101ELHL, U17 A1101ELHL, U18 A1101ELHL, U19 A1101ELHL, U2 A1101ELHL, U20 A1101ELHL, U21 A1101ELHL, U22 A1101ELHL, U23 A1101ELHL, U24 A1101ELHL, U25 A1101ELHL, U26 A1101ELHL, U27 A1101ELHL, U28 A1101ELHL, U29 A1101ELHL, U3 A1101ELHL, U30 A1101ELHL, U31 A1101ELHL, U32 A1101ELHL, U33 A1101ELHL, U34 A1101ELHL, U35 A1101ELHL, U36 A1101ELHL, U37 A1101ELHL, U38 A1101ELHL, U39 A1101ELHL, U4 A1101ELHL, U40 A1101ELHL, U41 A1101ELHL, U42 A1101ELHL, U43 A1101ELHL, U44 A1101ELHL, U45 A1101ELHL, U46 A1101ELHL, U47 A1101ELHL, U48 A1101ELHL, U49 A1101ELHL, U5 A1101ELHL, U50 A1101ELHL, U51 A1101ELHL, U52 A1101ELHL, U53 A1101ELHL, U54 A1101ELHL, U55 A1101ELHL, U56 A1101ELHL, U57 A1101ELHL, U58 A1101ELHL, U59 A1101ELHL, U6 A1101ELHL, U60 A1101ELHL, U61 A1101ELHL, U62 A1101ELHL, U63 A1101ELHL, U64 A1101ELHL, U65 A1101ELHL, U66 A1101ELHL, U67 A1101ELHL, U68 A1101ELHL, U7 A1101ELHL, U8 A1101ELHL, U9 A1101ELHL

Commit message: refactor readme file and remove old things
Parts:
- added AMUX0: CD74HC4067SM, Package_SO:SSOP-24_5.3x8.2mm_P0.65mm, B.Cu at (82.1, 70.7)
- added AMUX1: CD74HC4067SM, Package_SO:SSOP-24_5.3x8.2mm_P0.65mm, B.Cu at (145.0, 70.7)
- added AMUX2: CD74HC4067SM, Package_SO:SSOP-24_5.3x8.2mm_P0.65mm, B.Cu at (207.6, 68.6)
- added FID1: Fiducial, Fiducial:Fiducial_1mm_Mask3mm, F.Cu at (35.2, 121.0)
- added FID2: Fiducial, Fiducial:Fiducial_1mm_Mask3mm, F.Cu at (51.9, 35.7)
- added FID3: Fiducial, Fiducial:Fiducial_1mm_Mask3mm, F.Cu at (334.3, 97.6)
Connections:
- U1 pad 1: unconnected-(U1-VCC-Pad1) -> +3.3VA
- U1 pad 2: unconnected-(U1-VOUT-Pad2) -> /AMUX0:10
- U1 pad 3: unconnected-(U1-GND-Pad3) -> GND
- U10 pad 1: unconnected-(U10-VCC-Pad1) -> +3.3VA
- U10 pad 3: unconnected-(U10-GND-Pad3) -> GND
- U11 pad 1: unconnected-(U11-VCC-Pad1) -> +3.3VA
- U11 pad 3: unconnected-(U11-GND-Pad3) -> GND
- U12 pad 1: unconnected-(U12-VCC-Pad1) -> +3.3VA
- U12 pad 3: unconnected-(U12-GND-Pad3) -> GND
- U13 pad 1: unconnected-(U13-VCC-Pad1) -> +3.3VA
- U13 pad 3: unconnected-(U13-GND-Pad3) -> GND
- U14 pad 1: unconnected-(U14-VCC-Pad1) -> +3.3VA
- U14 pad 3: unconnected-(U14-GND-Pad3) -> GND
- U15 pad 1: unconnected-(U15-VCC-Pad1) -> +3.3VA
- U15 pad 3: unconnected-(U15-GND-Pad3) -> GND
- U16 pad 1: unconnected-(U16-VCC-Pad1) -> +3.3VA
- U16 pad 2: unconnected-(U16-VOUT-Pad2) -> /AMUX0:11
- U16 pad 3: unconnected-(U16-GND-Pad3) -> GND
- U17 pad 1: unconnected-(U17-VCC-Pad1) -> +3.3VA
- U17 pad 2: unconnected-(U17-VOUT-Pad2) -> /AMUX0:9
- U17 pad 3: unconnected-(U17-GND-Pad3) -> GND
- U18 pad 1: unconnected-(U18-VCC-Pad1) -> +3.3VA
- U18 pad 2: unconnected-(U18-VOUT-Pad2) -> /AMUX0:6
- U18 pad 3: unconnected-(U18-GND-Pad3) -> GND
- U19 pad 1: unconnected-(U19-VCC-Pad1) -> +3.3VA
- U19 pad 2: unconnected-(U19-VOUT-Pad2) -> /AMUX0:4
- U19 pad 3: unconnected-(U19-GND-Pad3) -> GND
- U2 pad 1: unconnected-(U2-VCC-Pad1) -> +3.3VA
- U2 pad 2: unconnected-(U2-VOUT-Pad2) -> /AMUX0:8
- U2 pad 3: unconnected-(U2-GND-Pad3) -> GND
- U20 pad 1: unconnected-(U20-VCC-Pad1) -> +3.3VA
- U20 pad 2: unconnected-(U20-VOUT-Pad2) -> /AMUX1:10
- U20 pad 3: unconnected-(U20-GND-Pad3) -> GND
- U21 pad 1: unconnected-(U21-VCC-Pad1) -> +3.3VA
- U21 pad 2: unconnected-(U21-VOUT-Pad2) -> /AMUX1:7
- U21 pad 3: unconnected-(U21-GND-Pad3) -> GND
- U22 pad 1: unconnected-(U22-VCC-Pad1) -> +3.3VA
- U22 pad 2: unconnected-(U22-VOUT-Pad2) -> /AMUX1:5
- U22 pad 3: unconnected-(U22-GND-Pad3) -> GND
- U23 pad 1: unconnected-(U23-VCC-Pad1) -> +3.3VA
- U23 pad 2: unconnected-(U23-VOUT-Pad2) -> /AMUX2:11
- U23 pad 3: unconnected-(U23-GND-Pad3) -> GND
- U24 pad 1: unconnected-(U24-VCC-Pad1) -> +3.3VA
- U24 pad 2: unconnected-(U24-VOUT-Pad2) -> /AMUX2:8
- U24 pad 3: unconnected-(U24-GND-Pad3) -> GND
- U25 pad 1: unconnected-(U25-VCC-Pad1) -> +3.3VA
- U25 pad 3: unconnected-(U25-GND-Pad3) -> GND
- U26 pad 1: unconnected-(U26-VCC-Pad1) -> +3.3VA
- U26 pad 3: unconnected-(U26-GND-Pad3) -> GND
- U27 pad 1: unconnected-(U27-VCC-Pad1) -> +3.3VA
- U27 pad 3: unconnected-(U27-GND-Pad3) -> GND
- U28 pad 1: unconnected-(U28-VCC-Pad1) -> +3.3VA
- U28 pad 3: unconnected-(U28-GND-Pad3) -> GND
- U29 pad 1: unconnected-(U29-VCC-Pad1) -> +3.3VA
- U29 pad 3: unconnected-(U29-GND-Pad3) -> GND
- U3 pad 1: unconnected-(U3-VCC-Pad1) -> +3.3VA
- U3 pad 2: unconnected-(U3-VOUT-Pad2) -> /AMUX0:7
- U3 pad 3: unconnected-(U3-GND-Pad3) -> GND
- U30 pad 1: unconnected-(U30-VCC-Pad1) -> +3.3VA
- U30 pad 3: unconnected-(U30-GND-Pad3) -> GND
- U31 pad 1: unconnected-(U31-VCC-Pad1) -> +3.3VA
- U31 pad 2: unconnected-(U31-VOUT-Pad2) -> /AMUX0:12
- U31 pad 3: unconnected-(U31-GND-Pad3) -> GND
- U32 pad 1: unconnected-(U32-VCC-Pad1) -> +3.3VA
- U32 pad 2: unconnected-(U32-VOUT-Pad2) -> /AMUX0:13
- U32 pad 3: unconnected-(U32-GND-Pad3) -> GND
- U33 pad 1: unconnected-(U33-VCC-Pad1) -> +3.3VA
- U33 pad 2: unconnected-(U33-VOUT-Pad2) -> /AMUX0:3
- U33 pad 3: unconnected-(U33-GND-Pad3) -> GND
- U34 pad 1: unconnected-(U34-VCC-Pad1) -> +3.3VA
- U34 pad 2: unconnected-(U34-VOUT-Pad2) -> /AMUX1:11
- U34 pad 3: unconnected-(U34-GND-Pad3) -> GND
- U35 pad 1: unconnected-(U35-VCC-Pad1) -> +3.3VA
- U35 pad 2: unconnected-(U35-VOUT-Pad2) -> /AMUX1:14
- U35 pad 3: unconnected-(U35-GND-Pad3) -> GND
- U36 pad 1: unconnected-(U36-VCC-Pad1) -> +3.3VA
- U36 pad 2: unconnected-(U36-VOUT-Pad2) -> /AMUX1:1
- U36 pad 3: unconnected-(U36-GND-Pad3) -> GND
- U37 pad 1: unconnected-(U37-VCC-Pad1) -> +3.3VA
- U37 pad 2: unconnected-(U37-VOUT-Pad2) -> /AMUX1:4
- U37 pad 3: unconnected-(U37-GND-Pad3) -> GND
- U38 pad 1: unconnected-(U38-VCC-Pad1) -> +3.3VA
- U38 pad 2: unconnected-(U38-VOUT-Pad2) -> /AMUX2:12
- U38 pad 3: unconnected-(U38-GND-Pad3) -> GND
- U39 pad 1: unconnected-(U39-VCC-Pad1) -> +3.3VA
- U39 pad 3: unconnected-(U39-GND-Pad3) -> GND
- U4 pad 1: unconnected-(U4-VCC-Pad1) -> +3.3VA
- U4 pad 2: unconnected-(U4-VOUT-Pad2) -> /AMUX0:5
- U4 pad 3: unconnected-(U4-GND-Pad3) -> GND
- U40 pad 1: unconnected-(U40-VCC-Pad1) -> +3.3VA
- U40 pad 3: unconnected-(U40-GND-Pad3) -> GND
- U41 pad 1: unconnected-(U41-VCC-Pad1) -> +3.3VA
- U41 pad 3: unconnected-(U41-GND-Pad3) -> GND
- U42 pad 1: unconnected-(U42-VCC-Pad1) -> +3.3VA
- U42 pad 3: unconnected-(U42-GND-Pad3) -> GND
- U43 pad 1: unconnected-(U43-VCC-Pad1) -> +3.3VA
- U43 pad 3: unconnected-(U43-GND-Pad3) -> GND
- U44 pad 1: unconnected-(U44-VCC-Pad1) -> +3.3VA
- U44 pad 3: unconnected-(U44-GND-Pad3) -> GND
- U45 pad 1: unconnected-(U45-VCC-Pad1) -> +3.3VA
- U45 pad 2: unconnected-(U45-VOUT-Pad2) -> /AMUX0:14
- U45 pad 3: unconnected-(U45-GND-Pad3) -> GND
- U46 pad 1: unconnected-(U46-VCC-Pad1) -> +3.3VA
- U46 pad 2: unconnected-(U46-VOUT-Pad2) -> /AMUX0:0
- U46 pad 3: unconnected-(U46-GND-Pad3) -> GND
- U47 pad 1: unconnected-(U47-VCC-Pad1) -> +3.3VA
- U47 pad 2: unconnected-(U47-VOUT-Pad2) -> /AMUX0:2
- U47 pad 3: unconnected-(U47-GND-Pad3) -> GND
- U48 pad 1: unconnected-(U48-VCC-Pad1) -> +3.3VA
- U48 pad 2: unconnected-(U48-VOUT-Pad2) -> /AMUX1:13
- U48 pad 3: unconnected-(U48-GND-Pad3) -> GND
- U49 pad 1: unconnected-(U49-VCC-Pad1) -> +3.3VA
- U49 pad 2: unconnected-(U49-VOUT-Pad2) -> /AMUX1:15
- U49 pad 3: unconnected-(U49-GND-Pad3) -> GND
- U5 pad 1: unconnected-(U5-VCC-Pad1) -> +3.3VA
- U5 pad 2: unconnected-(U5-VOUT-Pad2) -> /AMUX1:9
- U5 pad 3: unconnected-(U5-GND-Pad3) -> GND
- U50 pad 1: unconnected-(U50-VCC-Pad1) -> +3.3VA
- U50 pad 2: unconnected-(U50-VOUT-Pad2) -> /AMUX1:2
- U50 pad 3: unconnected-(U50-GND-Pad3) -> GND
- U51 pad 1: unconnected-(U51-VCC-Pad1) -> +3.3VA
- U51 pad 2: unconnected-(U51-VOUT-Pad2) -> /AMUX1:3
- U51 pad 3: unconnected-(U51-GND-Pad3) -> GND
- U52 pad 1: unconnected-(U52-VCC-Pad1) -> +3.3VA
- U52 pad 2: unconnected-(U52-VOUT-Pad2) -> /AMUX2:14
- U52 pad 3: unconnected-(U52-GND-Pad3) -> GND
- U53 pad 1: unconnected-(U53-VCC-Pad1) -> +3.3VA
- U53 pad 3: unconnected-(U53-GND-Pad3) -> GND
- U54 pad 1: unconnected-(U54-VCC-Pad1) -> +3.3VA
- U54 pad 3: unconnected-(U54-GND-Pad3) -> GND
- U55 pad 1: unconnected-(U55-VCC-Pad1) -> +3.3VA
- U55 pad 3: unconnected-(U55-GND-Pad3) -> GND
- U56 pad 1: unconnected-(U56-VCC-Pad1) -> +3.3VA
- U56 pad 3: unconnected-(U56-GND-Pad3) -> GND
- U57 pad 1: unconnected-(U57-VCC-Pad1) -> +3.3VA
- U57 pad 3: unconnected-(U57-GND-Pad3) -> GND
- U58 pad 1: unconnected-(U58-VCC-Pad1) -> +3.3VA
- U58 pad 2: unconnected-(U58-VOUT-Pad2) -> /AMUX0:15
- U58 pad 3: unconnected-(U58-GND-Pad3) -> GND
- U59 pad 1: unconnected-(U59-VCC-Pad1) -> +3.3VA
- U59 pad 2: unconnected-(U59-VOUT-Pad2) -> /AMUX0:1
- U59 pad 3: unconnected-(U59-GND-Pad3) -> GND
- U6 pad 1: unconnected-(U6-VCC-Pad1) -> +3.3VA
- U6 pad 2: unconnected-(U6-VOUT-Pad2) -> /AMUX1:8
- U6 pad 3: unconnected-(U6-GND-Pad3) -> GND
- U60 pad 1: unconnected-(U60-VCC-Pad1) -> +3.3VA
- U60 pad 2: unconnected-(U60-VOUT-Pad2) -> /AMUX1:12
- U60 pad 3: unconnected-(U60-GND-Pad3) -> GND
- U61 pad 1: unconnected-(U61-VCC-Pad1) -> +3.3VA
- U61 pad 2: unconnected-(U61-VOUT-Pad2) -> /AMUX1:0
- U61 pad 3: unconnected-(U61-GND-Pad3) -> GND
- U62 pad 1: unconnected-(U62-VCC-Pad1) -> +3.3VA
- U62 pad 2: unconnected-(U62-VOUT-Pad2) -> /AMUX2:13
- U62 pad 3: unconnected-(U62-GND-Pad3) -> GND
- U63 pad 1: unconnected-(U63-VCC-Pad1) -> +3.3VA
- U63 pad 2: unconnected-(U63-VOUT-Pad2) -> /AMUX2:15
- U63 pad 3: unconnected-(U63-GND-Pad3) -> GND
- U64 pad 1: unconnected-(U64-VCC-Pad1) -> +3.3VA
- U64 pad 3: unconnected-(U64-GND-Pad3) -> GND
- U65 pad 1: unconnected-(U65-VCC-Pad1) -> +3.3VA
- U65 pad 3: unconnected-(U65-GND-Pad3) -> GND
- U66 pad 1: unconnected-(U66-VCC-Pad1) -> +3.3VA
- U66 pad 3: unconnected-(U66-GND-Pad3) -> GND
- U67 pad 1: unconnected-(U67-VCC-Pad1) -> +3.3VA
- U67 pad 3: unconnected-(U67-GND-Pad3) -> GND
- U68 pad 1: unconnected-(U68-VCC-Pad1) -> +3.3VA
- U68 pad 3: unconnected-(U68-GND-Pad3) -> GND
- U7 pad 1: unconnected-(U7-VCC-Pad1) -> +3.3VA
- U7 pad 2: unconnected-(U7-VOUT-Pad2) -> /AMUX1:6
- U7 pad 3: unconnected-(U7-GND-Pad3) -> GND
- U8 pad 1: unconnected-(U8-VCC-Pad1) -> +3.3VA
- U8 pad 2: unconnected-(U8-VOUT-Pad2) -> /AMUX2:10
- U8 pad 3: unconnected-(U8-GND-Pad3) -> GND
- U9 pad 1: unconnected-(U9-VCC-Pad1) -> +3.3VA
- U9 pad 2: unconnected-(U9-VOUT-Pad2) -> /AMUX2:9
- U9 pad 3: unconnected-(U9-GND-Pad3) -> GND
Routing:
- net +3.3VA: track 0.00 -> 798.7 mm
- net /AMUX1:12: track 0.00 -> 57.5 mm
- net /AMUX2:13: track 0.00 -> 55.4 mm
- net /AMUX0:10: track 0.00 -> 51.0 mm
- net /AMUX0:1: track 0.00 -> 49.6 mm
- net /AMUX2:15: track 0.00 -> 47.5 mm
- net /AMUX1:0: track 0.00 -> 46.6 mm
- net /AMUX0:15: track 0.00 -> 46.3 mm
- net /AMUX1:3: track 0.00 -> 44.9 mm
- net /AMUX0:11: track 0.00 -> 43.4 mm
- net /AMUX0:12: track 0.00 -> 41.1 mm
- net /AMUX0:5: track 0.00 -> 40.5 mm
- net /AMUX2:10: track 0.00 -> 39.6 mm
- net /AMUX1:9: track 0.00 -> 38.8 mm
- net /AMUX1:6: track 0.00 -> 36.1 mm
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- added copper zone on B.Cu, net GND
- added copper zone on F.Cu, net GND
