File: kicad_2/kicad_2.kicad_sch (KiCad schematic)
At the start: 68 parts, among them U1 A1101ELHL, U10 A1101ELHL, U11 A1101ELHL, U12 A1101ELHL, U13 A1101ELHL, U14 A1101ELHL, U15 A1101ELHL, U16 A1101ELHL, U17 A1101ELHL, U18 A1101ELHL, U19 A1101ELHL, U2 A1101ELHL, U20 A1101ELHL, U21 A1101ELHL, U22 A1101ELHL, U23 A1101ELHL, U24 A1101ELHL, U25 A1101ELHL, U26 A1101ELHL, U27 A1101ELHL, U28 A1101ELHL, U29 A1101ELHL, U3 A1101ELHL, U30 A1101ELHL, U31 A1101ELHL, U32 A1101ELHL, U33 A1101ELHL, U34 A1101ELHL, U35 A1101ELHL, U36 A1101ELHL, U37 A1101ELHL, U38 A1101ELHL, U39 A1101ELHL, U4 A1101ELHL, U40 A1101ELHL, U41 A1101ELHL, U42 A1101ELHL, U43 A1101ELHL, U44 A1101ELHL, U45 A1101ELHL, U46 A1101ELHL, U47 A1101ELHL, U48 A1101ELHL, U49 A1101ELHL, U5 A1101ELHL, U50 A1101ELHL, U51 A1101ELHL, U52 A1101ELHL, U53 A1101ELHL, U54 A1101ELHL, U55 A1101ELHL, U56 A1101ELHL, U57 A1101ELHL, U58 A1101ELHL, U59 A1101ELHL, U6 A1101ELHL, U60 A1101ELHL, U61 A1101ELHL, U62 A1101ELHL, U63 A1101ELHL, U64 A1101ELHL, U65 A1101ELHL, U66 A1101ELHL, U67 A1101ELHL, U68 A1101ELHL, U7 A1101ELHL, U8 A1101ELHL, U9 A1101ELHL

Commit message: refactor readme file and remove old things
Parts:
- added AMUX0, AMUX1, AMUX2: CD74HC4067SM, Package_SO:SSOP-24_5.3x8.2mm_P0.65mm, symbol 74xx:CD74HC4067SM
- added FID1, FID2, FID3: Fiducial, Fiducial:Fiducial_1mm_Mask3mm, symbol Mechanical:Fiducial
Connections:
- net +3.3VA: now reaches U25.1 (VCC)
- net +3.3VA: now also U1.1 (VCC), U10.1 (VCC), U11.1 (VCC), U12.1 (VCC), U13.1 (VCC), U14.1 (VCC), U15.1 (VCC), U16.1 (VCC), U17.1 (VCC), U18.1 (VCC), U19.1 (VCC), U2.1 (VCC), U20.1 (VCC), U21.1 (VCC), U22.1 (VCC), U23.1 (VCC), U24.1 (VCC), U26.1 (VCC), U27.1 (VCC), U28.1 (VCC), U29.1 (VCC), U3.1 (VCC), U30.1 (VCC), U31.1 (VCC), U32.1 (VCC), U33.1 (VCC), U34.1 (VCC), U35.1 (VCC), U36.1 (VCC), U37.1 (VCC), U38.1 (VCC), U39.1 (VCC), U4.1 (VCC), U40.1 (VCC), U41.1 (VCC), U42.1 (VCC), U43.1 (VCC), U44.1 (VCC), U45.1 (VCC), U46.1 (VCC), U47.1 (VCC), U48.1 (VCC), U49.1 (VCC), U5.1 (VCC), U50.1 (VCC), U51.1 (VCC), U52.1 (VCC), U53.1 (VCC), U54.1 (VCC), U55.1 (VCC), U56.1 (VCC), U57.1 (VCC), U58.1 (VCC), U59.1 (VCC), U6.1 (VCC), U60.1 (VCC), U61.1 (VCC), U62.1 (VCC), U63.1 (VCC), U64.1 (VCC), U65.1 (VCC), U66.1 (VCC), U67.1 (VCC), U68.1 (VCC), U7.1 (VCC), U8.1 (VCC), U9.1 (VCC), AMUX0.24 (VCC), AMUX1.24 (VCC), AMUX2.24 (VCC)
- net GND: now reaches U25.3 (GND)
- net GND: now also U1.3 (GND), U10.3 (GND), U11.3 (GND), U12.3 (GND), U13.3 (GND), U14.3 (GND), U15.3 (GND), U16.3 (GND), U17.3 (GND), U18.3 (GND), U19.3 (GND), U2.3 (GND), U20.3 (GND), U21.3 (GND), U22.3 (GND), U23.3 (GND), U24.3 (GND), U26.3 (GND), U27.3 (GND), U28.3 (GND), U29.3 (GND), U3.3 (GND), U30.3 (GND), U31.3 (GND), U32.3 (GND), U33.3 (GND), U34.3 (GND), U35.3 (GND), U36.3 (GND), U37.3 (GND), U38.3 (GND), U39.3 (GND), U4.3 (GND), U40.3 (GND), U41.3 (GND), U42.3 (GND), U43.3 (GND), U44.3 (GND), U45.3 (GND), U46.3 (GND), U47.3 (GND), U48.3 (GND), U49.3 (GND), U5.3 (GND), U50.3 (GND), U51.3 (GND), U52.3 (GND), U53.3 (GND), U54.3 (GND), U55.3 (GND), U56.3 (GND), U57.3 (GND), U58.3 (GND), U59.3 (GND), U6.3 (GND), U60.3 (GND), U61.3 (GND), U62.3 (GND), U63.3 (GND), U64.3 (GND), U65.3 (GND), U66.3 (GND), U67.3 (GND), U68.3 (GND), U7.3 (GND), U8.3 (GND), U9.3 (GND), AMUX0.12 (GND), AMUX0.15 (~{E}), AMUX1.12 (GND), AMUX1.15 (~{E}), AMUX2.12 (GND), AMUX2.15 (~{E})
- net AMUX1:4: now reaches U37.2 (VOUT)
- net AMUX1:4: now also AMUX1.5 (I4)
- net AMUX0:4: now reaches U19.2 (VOUT)
- net AMUX0:4: now also AMUX0.5 (I4)
- net AMUX1:13: now reaches U48.2 (VOUT)
- net AMUX1:13: now also AMUX1.18 (I13)
- net AMUX1:11: now reaches U34.2 (VOUT)
- net AMUX1:11: now also AMUX1.20 (I11)
- net AMUX0:6: now reaches U18.2 (VOUT)
- net AMUX0:6: now also AMUX0.3 (I6)
- net AMUX0:7: now reaches U3.2 (VOUT)
- net AMUX0:7: now also AMUX0.2 (I7)
- net AMUX0:8: now reaches U2.2 (VOUT)
- net AMUX0:8: now also AMUX0.23 (I8)
- net AMUX2:13: now reaches U62.2 (VOUT)
- net AMUX2:13: now also AMUX2.18 (I13)
- net AMUX2:15: now reaches U63.2 (VOUT)
- net AMUX2:15: now also AMUX2.16 (I15)
- net AMUX2:12: now reaches U38.2 (VOUT)
- net AMUX2:12: now also AMUX2.19 (I12)
- net AMUX0:13: now reaches U32.2 (VOUT)
- net AMUX0:13: now also AMUX0.18 (I13)
- net AMUX2:11: now reaches U23.2 (VOUT)
- net AMUX2:11: now also AMUX2.20 (I11)
- net AMUX1:10: now reaches U20.2 (VOUT)
- net AMUX1:10: now also AMUX1.21 (I10)
- net AMUX2:8: now reaches U24.2 (VOUT)
- net AMUX2:8: now also AMUX2.23 (I8)
- net AMUX2:10: now reaches U8.2 (VOUT)
- net AMUX2:10: now also AMUX2.21 (I10)
- net AMUX0:0: now reaches U46.2 (VOUT)
- net AMUX0:0: now also AMUX0.9 (I0)
- net AMUX1:8: now reaches U6.2 (VOUT)
- net AMUX1:8: now also AMUX1.23 (I8)
- net AMUX0:11: now reaches U16.2 (VOUT)
- net AMUX0:11: now also AMUX0.20 (I11)
- net AMUX0:15: now reaches U58.2 (VOUT)
- net AMUX0:15: now also AMUX0.16 (I15)
- net AMUX0:5: now reaches U4.2 (VOUT)
- net AMUX0:5: now also AMUX0.4 (I5)
- net AMUX0:10: now reaches U1.2 (VOUT)
- net AMUX0:10: now also AMUX0.21 (I10)
- net AMUX0:12: now reaches U31.2 (VOUT)
- net AMUX0:12: now also AMUX0.19 (I12)
- net AMUX1:12: now reaches U60.2 (VOUT)
- net AMUX1:12: now also AMUX1.19 (I12)
- net AMUX0:14: now reaches U45.2 (VOUT)
- net AMUX0:14: now also AMUX0.17 (I14)
- net AMUX1:5: now reaches U22.2 (VOUT)
- net AMUX1:5: now also AMUX1.4 (I5)
- net AMUX1:15: now reaches U49.2 (VOUT)
- net AMUX1:15: now also AMUX1.16 (I15)
- net AMUX1:2: now reaches U50.2 (VOUT)
- net AMUX1:2: now also AMUX1.7 (I2)
- net AMUX1:1: now reaches U36.2 (VOUT)
- net AMUX1:1: now also AMUX1.8 (I1)
- net AMUX0:2: now reaches U47.2 (VOUT)
- net AMUX0:2: now also AMUX0.7 (I2)
- net AMUX1:6: now reaches U7.2 (VOUT)
- net AMUX1:6: now also AMUX1.3 (I6)
- net AMUX1:3: now reaches U51.2 (VOUT)
- net AMUX1:3: now also AMUX1.6 (I3)
- net AMUX1:9: now reaches U5.2 (VOUT)
- net AMUX1:9: now also AMUX1.22 (I9)
- net AMUX2:14: now reaches U52.2 (VOUT)
- net AMUX2:14: now also AMUX2.17 (I14)
- net AMUX2:9: now reaches U9.2 (VOUT)
- net AMUX2:9: now also AMUX2.22 (I9)
- net AMUX1:7: now reaches U21.2 (VOUT)
- net AMUX1:7: now also AMUX1.2 (I7)
- net AMUX0:1: now reaches U59.2 (VOUT)
- net AMUX0:1: now also AMUX0.8 (I1)
- net AMUX1:0: now reaches U61.2 (VOUT)
- net AMUX1:0: now also AMUX1.9 (I0)
- net AMUX0:3: now reaches U33.2 (VOUT)
- net AMUX0:3: now also AMUX0.6 (I3)
- net AMUX1:14: now reaches U35.2 (VOUT)
- net AMUX1:14: now also AMUX1.17 (I14)
- net AMUX0:9: now reaches U17.2 (VOUT)
- net AMUX0:9: now also AMUX0.22 (I9)
- new net ADC0: AMUX0.1 (COM)
- new net ADC1: AMUX1.1 (COM)
- new net ADC2: AMUX2.1 (COM)
- new net AMUX2:0: AMUX2.9 (I0)
- new net AMUX2:1: AMUX2.8 (I1)
- new net AMUX2:2: AMUX2.7 (I2)
- new net AMUX2:3: AMUX2.6 (I3)
- new net AMUX2:4: AMUX2.5 (I4)
- new net AMUX2:5: AMUX2.4 (I5)
- new net AMUX2:6: AMUX2.3 (I6)
- new net AMUX2:7: AMUX2.2 (I7)
- new net SELECT0: AMUX0.10 (S0), AMUX1.10 (S0), AMUX2.10 (S0)
- new net SELECT1: AMUX0.11 (S1), AMUX1.11 (S1), AMUX2.11 (S1)
- new net SELECT2: AMUX0.14 (S2), AMUX1.14 (S2), AMUX2.14 (S2)
- new net SELECT3: AMUX0.13 (S3), AMUX1.13 (S3), AMUX2.13 (S3)
Other:
- moved on the sheet: U10, U11, U12, U13, U14, U15, U16, U17, U18, U19, U2, U20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
