File: kicad/Rev 2.0/layout_board/layout_board.kicad_pcb (KiCad board)
At the start: 2 copper layers, 309.6 x 95.2 mm, 150 parts, among them J1 Conn_01x11_Socket, U0:0 GH39FKSW, U0:1 GH39FKSW, U0:10 GH39FKSW, U0:11 GH39FKSW, U0:12 GH39FKSW, U0:13 GH39FKSW, U0:14 GH39FKSW, U0:2 GH39FKSW, U0:3 GH39FKSW, U0:4 GH39FKSW, U0:5 GH39FKSW, U0:6 GH39FKSW, U0:7 GH39FKSW, U0:8 GH39FKSW, U0:9 GH39FKSW, U1 CD4067BPWR, U1:0 GH39FKSW, U1:1 GH39FKSW, U1:10 GH39FKSW, U1:11 GH39FKSW, U1:12 GH39FKSW, U1:13 GH39FKSW, U1:14 GH39FKSW, U1:2 GH39FKSW, U1:3 GH39FKSW, U1:4 GH39FKSW, U1:5 GH39FKSW, U1:6 GH39FKSW, U1:7 GH39FKSW, U1:8 GH39FKSW, U1:9 GH39FKSW, U2 CD4067BPWR, U2:0 GH39FKSW, U2:1 GH39FKSW, U2:10 GH39FKSW, U2:11 GH39FKSW, U2:12 GH39FKSW, U2:13 GH39FKSW, U2:2 GH39FKSW, U2:3 GH39FKSW, U2:4 GH39FKSW, U2:5 GH39FKSW, U2:6 GH39FKSW, U2:7 GH39FKSW, U2:8 GH39FKSW, U2:9 GH39FKSW, U3 CD4067BPWR, U3:1 GH39FKSW, U3:10 GH39FKSW, U3:11 GH39FKSW, U3:12 GH39FKSW, U3:13 GH39FKSW, U3:2 GH39FKSW, U3:3 GH39FKSW, U3:4 GH39FKSW, U3:5 GH39FKSW, U3:6 GH39FKSW, U3:7 GH39FKSW, U3:8 GH39FKSW, U3:9 GH39FKSW, U4 CD4067BPWR, U4:1 GH39FKSW, U4:10 GH39FKSW, U4:12 GH39FKSW, U4:13 GH39FKSW, U4:14 GH39FKSW, U4:2 GH39FKSW, U4:3 GH39FKSW, U4:5 GH39FKSW, U4:7 GH39FKSW, U4:9 GH39FKSW, U5 CD4067BPWR

Commit message: wip: remove flex pcb
Parts:
- added REF**: SolderWirePad_1x01_SMD_1x2mm, Connector_Wire:SolderWirePad_1x01_SMD_1x2mm, F.Cu at (49.4, 39.6)
- added REF**: MountingHole_2.2mm_M2, MountingHole:MountingHole_2.2mm_M2, F.Cu at (121.9, -2.83)
- J1: value Conn_01x11_Socket -> HC-FPC-05-10-12RLTAG; footprint Custom:Flex Cable connector -> JLCPCB:FPC-SMD_12P-P0.50_HCTL_HC-FPC-05-10-12RLTAG
- moved J1 0.75 mm to (53.1, 34.3), turned to 90 degrees
Connections:
- J1 pad 1: /SELECT3 -> GND
- J1 pad 10: /ADC0 -> /SELECT1
- J1 pad 11: GND -> /SELECT2
- J1 pad 2: /SELECT2 -> /ADC0
- J1 pad 3: /SELECT1 -> /ADC1
- J1 pad 4: /SELECT0 -> /ADC2
- J1 pad 5: +3.3VA -> /ADC3
- J1 pad 7: /ADC3 -> GND
- J1 pad 8: /ADC2 -> +3.3VA
- J1 pad 9: /ADC1 -> /SELECT0
Routing:
- net +3.3VA: track 2002.6 -> 1997.8 mm, vias 50 -> 52
- net /SELECT1: track 300.6 -> 299.8 mm
- net /SELECT3: track 304.1 -> 303.3 mm
- net /SELECT0: track 302.7 -> 301.9 mm
- net /SELECT2: track 307.6 -> 306.7 mm
- net /ADC0: track 31.7 -> 31.1 mm
- net /ADC4: track 262.5 -> 261.9 mm
- net /ADC3: track 204.8 -> 204.2 mm
- net /ADC1: track 89.7 -> 89.1 mm
- net /ADC2: track 147.0 -> 146.4 mm
- net GND: vias 3251 -> 3253
Other:
- outline, holes or cut-outs redrawn

Commit message: wip: add logo and qrcode
Parts:
- added REF**: MountingHole_3.2mm_M3_ISO7380_Pad_TopOnly, MountingHole:MountingHole_3.2mm_M3_ISO7380_Pad_TopOnly, B.Cu at (105.6, 86.6)
- added REF**: MountingHole_3.2mm_M3_ISO7380_Pad_TopOnly, MountingHole:MountingHole_3.2mm_M3_ISO7380_Pad_TopOnly, B.Cu at (319.1, 84.2)
- added REF**: MountingHole_3.2mm_M3_ISO7380_Pad_TopOnly, MountingHole:MountingHole_3.2mm_M3_ISO7380_Pad_TopOnly, B.Cu at (315.8, 49.7)
- added REF**: MountingHole_3.2mm_M3_ISO7380_Pad_TopOnly, MountingHole:MountingHole_3.2mm_M3_ISO7380_Pad_TopOnly, B.Cu at (40.5, 47.6)
- added REF**: MountingHole_3.2mm_M3_ISO7380_Pad_TopOnly, MountingHole:MountingHole_3.2mm_M3_ISO7380_Pad_TopOnly, B.Cu at (109.5, 39.0)
- added REF**: MountingHole_3.2mm_M3_ISO7380_Pad_TopOnly, MountingHole:MountingHole_3.2mm_M3_ISO7380_Pad_TopOnly, B.Cu at (44.1, 110.7)
- added REF**: MountingHole_3.2mm_M3_ISO7380_Pad_TopOnly, MountingHole:MountingHole_3.2mm_M3_ISO7380_Pad_TopOnly, B.Cu at (266.7, 104.2)
- added REF**: MountingHole_3.2mm_M3_ISO7380_Pad_TopOnly, MountingHole:MountingHole_3.2mm_M3_ISO7380_Pad_TopOnly, B.Cu at (214.3, 48.2)
- REF**: value MountingHole_2.2mm_M2 -> MountingHole_3.2mm_M3_ISO7380_Pad_TopOnly; footprint MountingHole:MountingHole_2.2mm_M2 -> MountingHole:MountingHole_3.2mm_M3_ISO7380_Pad_TopOnly; moved to B.Cu
- moved REF** 127.8 mm to (175.6, 113.1), turned to 180 degrees
Routing:
- net GND: vias 3253 -> 3204
