File: kicad/Rev 2.0/layout_board/layout_board.kicad_pcb (KiCad board)
At the start: 2 copper layers, 309.6 x 95.2 mm, 160 parts, among them J1 HC-FPC-05-10-12RLTAG, U0:0 GH39FKSW, U0:1 GH39FKSW, U0:10 GH39FKSW, U0:11 GH39FKSW, U0:12 GH39FKSW, U0:13 GH39FKSW, U0:14 GH39FKSW, U0:2 GH39FKSW, U0:3 GH39FKSW, U0:4 GH39FKSW, U0:5 GH39FKSW, U0:6 GH39FKSW, U0:7 GH39FKSW, U0:8 GH39FKSW, U0:9 GH39FKSW, U1 CD4067BPWR, U1:0 GH39FKSW, U1:1 GH39FKSW, U1:10 GH39FKSW, U1:11 GH39FKSW, U1:12 GH39FKSW, U1:13 GH39FKSW, U1:14 GH39FKSW, U1:2 GH39FKSW, U1:3 GH39FKSW, U1:4 GH39FKSW, U1:5 GH39FKSW, U1:6 GH39FKSW, U1:7 GH39FKSW, U1:8 GH39FKSW, U1:9 GH39FKSW, U2 CD4067BPWR, U2:0 GH39FKSW, U2:1 GH39FKSW, U2:10 GH39FKSW, U2:11 GH39FKSW, U2:12 GH39FKSW, U2:13 GH39FKSW, U2:2 GH39FKSW, U2:3 GH39FKSW, U2:4 GH39FKSW, U2:5 GH39FKSW, U2:6 GH39FKSW, U2:7 GH39FKSW, U2:8 GH39FKSW, U2:9 GH39FKSW, U3 CD4067BPWR, U3:1 GH39FKSW, U3:10 GH39FKSW, U3:11 GH39FKSW, U3:12 GH39FKSW, U3:13 GH39FKSW, U3:2 GH39FKSW, U3:3 GH39FKSW, U3:4 GH39FKSW, U3:5 GH39FKSW, U3:6 GH39FKSW, U3:7 GH39FKSW, U3:8 GH39FKSW, U3:9 GH39FKSW, U4 CD4067BPWR, U4:1 GH39FKSW, U4:10 GH39FKSW, U4:12 GH39FKSW, U4:13 GH39FKSW, U4:14 GH39FKSW, U4:2 GH39FKSW, U4:3 GH39FKSW, U4:5 GH39FKSW, U4:7 GH39FKSW, U4:9 GH39FKSW, U5 CD4067BPWR

Commit message: wip: daughter board done
Routing:
- net GND: vias 3204 -> 3210
Changed lines of the file:
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@@
 		(fp_arc
 			(start 9.03125 8.000001)
-			(mid 8.677729 7.853537)
+			(mid 8.677693 7.853543)
 			(end 8.53125 7.500001)
 			(stroke
@@
 		(fp_arc
 			(start 14.780039 -5.999999)
-			(mid 15.133567 -5.853539)
+			(mid 15.133602 -5.853545)
 			(end 15.280039 -5.499999)
 			(stroke
@@
 		(fp_arc
 			(start 15.28125 7.500001)
-			(mid 15.134806 7.853571)
+			(mid 15.1348 7.853536)
 			(end 14.78125 8.000001)
 			(stroke
@@
 		(fp_arc
 			(start 15.28125 7.500001)
-			(mid 15.134806 7.853571)
+			(mid 15.1348 7.853536)
 			(end 14.78125 8.000001)
 			(stroke
@@
 		(fp_arc
 			(start 14.780039 -5.999999)
-			(mid 15.133567 -5.853539)
+			(mid 15.133602 -5.853545)
 			(end 15.280039 -5.499999)
 			(stroke
@@
 		(fp_arc
 			(start 9.03125 8.000001)
-			(mid 8.677729 7.853537)
+			(mid 8.677693 7.853543)
 			(end 8.53125 7.500001)
 			(stroke
@@
 		(fp_arc
 			(start 15.28125 7.500001)
-			(mid 15.134806 7.853571)
+			(mid 15.1348 7.853536)
 			(end 14.78125 8.000001)
 			(stroke
@@
 		(fp_arc
 			(start 14.780039 -5.999999)
-			(mid 15.133567 -5.853539)
+			(mid 15.133602 -5.853545)
 			(end 15.280039 -5.499999)
 			(stroke
@@
 		(fp_arc
 			(start 9.03125 8.000001)
-			(mid 8.677729 7.853537)
+			(mid 8.677693 7.853543)
 			(end 8.53125 7.500001)
 			(stroke
@@
 		(fp_arc
 			(start 9.03125 8.000001)
-			(mid 8.677729 7.853537)
+			(mid 8.677693 7.853543)
 			(end 8.53125 7.500001)
 			(stroke
@@
 		(fp_arc
 			(start 14.780039 -5.999999)
-			(mid 15.133567 -5.853539)
+			(mid 15.133602 -5.853545)
 			(end 15.280039 -5.499999)
 			(stroke
@@
 		(fp_arc
 			(start 15.28125 7.500001)
-			(mid 15.134806 7.853571)
+			(mid 15.1348 7.853536)
 			(end 14.78125 8.000001)
 			(stroke
@@
 	)
 	(via
+		(at 51.420074 31.960813)
+		(size 0.7)
+		(drill 0.3)
+		(layers "F.Cu" "B.Cu")
+		(free yes)
+		(net 1)
+	)
+	(via
 		(at 121.210514 122.82286)
 		(size 0.7)
@@
 	)
 	(via
+		(at 52.945561 34.156026)
+		(size 0.7)
+		(drill 0.3)
+		(layers "F.Cu" "B.Cu")
+		(free yes)
+		(net 1)
+	)
+	(via
 		(at 133.498716 42.602015)
 		(size 0.7)
@@
 	)
 	(via
+		(at 52.982768 36.500067)
+		(size 0.7)
+		(drill 0.3)
+		(layers "F.Cu" "B.Cu")
+		(free yes)
+		(net 1)
+	)
+	(via
 		(at 199.950514 87.26286)
 		(size 0.7)
@@
 	)
 	(via
+		(at 51.382867 36.537274)
+		(size 0.7)
+		(drill 0.3)
+		(layers "F.Cu" "B.Cu")
+		(free yes)
+		(net 1)
+	)
+	(via
 		(at 188.121017 73.945179)
 		(size 0.7)
@@
 	)
 	(via
+		(at 53.094389 31.960813)
+		(size 0.7)
+		(drill 0.3)
+		(layers "F.Cu" "B.Cu")
+		(free yes)
+		(net 1)
+	)
+	(via
 		(at 255.830514 66.94286)
 		(size 0.7)
@@
 	)
 	(via
+		(at 51.457281 34.193233)
+		(size 0.7)
+		(drill 0.3)
+		(layers "F.Cu" "B.Cu")
+		(free yes)
+		(net 1)
+	)
+	(via
 		(at 128.830514 46.62286)
 		(size 0.7)
@@
 		(net 1)
 		(net_name "GND")
-		(layer "F.Cu")
-		(hatch edge 0.5)
-		(priority 1)
-		(connect_pads
-			(clearance 0.2)
-		)
-		(min_thickness 0.254)
-		(filled_areas_thickness no)
-		(fill yes
-			(thermal_gap 0.5)
-			(thermal_bridge_width 0.5)
-		)
-		(polygon
-			(pts
-				(xy 19.608089 21.319611) (xy 21.096369 132.568541) (xy 344.53682 132.568541) (xy 346.211135 22.993926)
-				(xy 19.645296 21.319611)
-			)
-		)
-	)
-	(zone
-		(net 0)
-		(net_name "")
-		(layers "F.Cu" "Edge.Cuts")
-		(hatch edge 0.5)
-		(connect_pads
-			(clearance 0)
-		)
-		(min_thickness 0.25)
-		(filled_areas_thickness no)
-		(keepout
-			(tracks allowed)
-			(vias allowed)
-			(pads allowed)
-			(copperpour not_allowed)
-			(footprints allowed)
-		)
-		(fill
-			(thermal_gap 0.5)
-			(thermal_bridge_width 0.5)
-		)
-		(polygon
-			(pts
-				(xy 51.47359 30.69528) (xy 52.424663 30.695775) (xy 52.424663 37.765105) (xy 51.47359 37.765105)
-			)
-		)
-	)
-	(zone
-		(net 1)
-		(net_name "GND")
-		(layer "B.Cu")
+		(layers "F&B.Cu")
 		(hatch edge 0.5)
 		(connect_pads

Commit message: wip: gerber files
Routing:
- net +3.3VA: track 1997.8 -> 2135.7 mm, vias 52 -> 68
- net GND: vias 3210 -> 3235

Commit message: wip: changing amuxes
Parts:
- U1, U2, U3, U4, U5: footprint JLCPCB:TSSOP-24_L7.8-W4.4-P0.65-LS6.4-BL_1 -> Custom:(T_S)SOP-24_5.3x8.2mm_P0.65mm
- turned U1 to 0 degrees
- turned U2 to 0 degrees
Routing:
- net /AMUX1:7: track 13.6 -> 14.3 mm
- net /AMUX0:0: track 9.08 -> 8.55 mm
- net GND: vias 3235 -> 3238
